File: Hardware/kitt_mb01/eagle/mb_01.sch (EAGLE design)
At the start: 58 parts, among them CON1 ARDUINO_UNO, IC2.00 BQ24266RGET, P1 JST.S2B-PH-SM4-TB

Commit message: entered motor controller circuitry
Parts:
- removed C1: 470uF, rcl:CPOL-EUSMCP
- removed C2: 390uF, rcl:CPOL-EUSMCP
- removed D2: MBRS320T3, diode:MBRS320T3
- removed L1: (no value), inductor-neosid:SM-B5
- removed LED1: LG_T679-E1F1-1, led:LG_T679-E1F1-1
- removed TP1: TPSQTP19SQ, testpad:TPSQTP19SQ
- removed X1: (no value), con-phoenix-254:MPT2
- added C1.01: 22uF/25V, rcl:C-EUC1210K
- added C1.02: 100nF, rcl:C-EUC0402K
- added C1.04: XX, rcl:C-EUC0402K
- added C1.05, C1.06: 22uF/6.3V, rcl:C-EUC1206K
- added C4.01: 47uF/25V, rcl:CPOL-EUC/6032-28R
- added C4.02: 100nF/25V, resistor:C-EUC0603K
- added C4.03: (no value), resistor:C-EUC0805K
- added C4.04, C4.05: 220nF/25V, rcl:C-EUC0603K
- added IC1: (no value), kitt.ic:DRV8871
- added IC1.01: RT8293A, kitt.ic:RT8293A
- added L2.01: 2.6uH, rcl:L-EUWE-TPC
- added L4.01: BEAD, inductors:BLM15HB121SN1
- added R1.03, R1.04: XX, rcl:R-EU_R0402
- added R1.05, R1.06: [0R], rcl:R-EU_R0402
- added R4.01, R4.02: [0R], rcl:R-EU_M0805
- added R4.03: 22kR, resistor:R-EU_R0402
- added R4.04, R4.05: 1kR, resistor:R-EU_R0402
- added RAILS, SOC, SOC1: (no value), con-phoenix-254:MPT2
- C1.03: value [*a]1uF -> 100nF; device rcl:C-EUC0805K -> rcl:C-EUC0402K
- L1.01: value 22uH -> BEAD; device rcl:L-EUWE-TPC -> inductors:BLM15HB121SN1
- L1.02: value 2.6uH -> 4.7uH
- L2: value (none) -> BEAD
- R1.01: value <1>??R -> 100kR; device rcl:R-EU_R0805 -> rcl:R-EU_R0402
- R1.02: value <2>??R -> XX; device rcl:R-EU_R0805 -> rcl:R-EU_R0402
Connections:
- net ARDUINO.SCL renamed SCL
- net ARDUINO.SDA renamed SDA
- net AU.!IRQ_GYRO renamed !IRQ_GYRO
- new net MOT.IN1: CON1G$3.IO.3, IC1.IN1, R4.05.2
- new net MOT.IN2: CON1G$3.IO.4, IC1.IN2, R4.04.2
- new net N$25: C1.04.1, IC1.01.COMP
- new net N$28: IC1.01.FB, R1.03.1, R1.04.2
- new net N$29: C1.05.1, C1.06.1, L1.02.1, L2.1, R1.03.2
- new net N$30: C1.03.2, IC1.01.SW, L1.02.2
- new net N$31: C1.03.1, IC1.01.BOOT
- new net N$32: L2.2, R1.05.2, R1.06.1
- new net N$33: C4.04.2, C4.05.1, IC1.OUT1, SOC1-1.1
- new net N$34: IC1.OUT2, R4.02.2
- new net N$35: IC1.ILIM, R4.03.2
- net +12V: now also C4.03.1, L4.01.2, R2.1
- net +4.1V: no longer R2.04.1
- net +5V: now also IC2.00PINS.IN@1, IC2.00PINS.IN@2, R1.05.1, R1.06.2, R2.02.2, SOC-1.1; no longer L2.2
- net GND: now also C1.01.2, C1.02.2, C1.05.2, C1.06.2, C4.01.-, C4.02.2, C4.03.2, C4.05.2, IC1.01.GND, IC1.01.PAD, IC1.GND, IC1.PAD, IC1.PGND, R1.02.1, R1.04.1, R4.01.1, R4.03.1, R4.04.1, R4.05.1, SOC-2.1; no longer C1.-, C1.03.2, C2.-, D2.A, R1.01.1
- net GNDA: now also RAILS-2.1; no longer X1-2.1
- net N$10: now also C4.01.+, C4.02.1, C4.04.1, IC1.VM, L4.01.1; no longer LED1.C, R2.1
- net N$12: now also L2.01.2; no longer L1.02.2
- net N$18: now also L2.01.1; no longer L1.02.1
- net N$2: now also L1.01.1; no longer L1.1
- net N$3: now also C1.01.1, IC1.01.VIN, L1.01.2, R1.01.1; no longer C1.+, L1.2
- net N$4: now also IC1.01.EN; no longer R1.02.1, TP1.TP
- net N$5: now also C1.02.1, IC1.01.SS; no longer D2.C, L1.01.2
- net N$7: now also C1.04.2; no longer C2.+, L1.01.1, L2.1
- net N$9: now also R4.01.2, R4.02.1, SOC1-2.1; no longer IC2.00PINS.IN@1, IC2.00PINS.IN@2, R2.02.2
- net V+: now also R2.04.1
- net VCC/2: now also RAILS-1.1; no longer LED1.A, X1-1.1
Other:
- note added: "KITT MB01 - Axis Sensor"
- note removed: "<1,2>: 5V=(1+<2>/<1>)*1.23V"
- note removed: "INSERT DC/DC HERE"
- note removed: "TODO: VDD_ALT_V"
- note removed: "The LED here is dual purpose: 1. Idicator for Rail Voltage 2. Reverse Polarity Protection for the SoC Board RX independent from the main power chain"

Commit message: began working on the fullbridge
Parts:
- L2: device inductor-neosid:SM-B5 -> inductors:BLM15HB121SN1
- renumbered U$1 to IC3.01
Changed lines of the file:
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@@
 <part name="L1.02" library="rcl" deviceset="L-EU" device="WE-TPC" value="4.7uH"/>
 <part name="P+5VMAIN" library="supply1" deviceset="+5V" device="" value="+5V-MAIN"/>
-<part name="L2" library="inductor-neosid" deviceset="SM-B" device="5" value="BEAD"/>
+<part name="L2" library="inductors" deviceset="BLM15H" device="" technology="B121SN1" value="BEAD"/>
 <part name="FRAME1" library="frames" deviceset="A4L-LOC" device=""/>
 <part name="FRAME2" library="frames" deviceset="A4L-LOC" device=""/>
@@
 <part name="P1" library="kitt.con" deviceset="JST.S2B-PH-SM4-TB" device=""/>
 <part name="REF5" library="kitt.refs" deviceset="REF.KITT-MB01" device=""/>
-<part name="U$1" library="kitt.ic" deviceset="LSM9DS1" device=""/>
+<part name="IC3.01" library="kitt.ic" deviceset="LSM9DS1" device=""/>
 <part name="FRAME4" library="frames" deviceset="A4L-LOC" device=""/>
 <part name="+3V1" library="supply1" deviceset="+3V3" device=""/>
@@
 <segment>
 <pinref part="L2" gate="G$1" pin="2"/>
-<wire x1="224.79" y1="143.51" x2="229.87" y2="143.51" width="0.1524" layer="91"/>
+<wire x1="227.33" y1="143.51" x2="229.87" y2="143.51" width="0.1524" layer="91"/>
 <pinref part="R1.05" gate="G$1" pin="2"/>
 <wire x1="229.87" y1="146.05" x2="229.87" y2="143.51" width="0.1524" layer="91"/>
@@
 </plain>
 <instances>
-<instance part="U$1" gate="G$1" x="127" y="114.3"/>
+<instance part="IC3.01" gate="G$1" x="127" y="114.3"/>
 <instance part="FRAME4" gate="G$1" x="0" y="0"/>
 <instance part="+3V1" gate="G$1" x="96.52" y="149.86"/>
@@
 <segment>
 <pinref part="+3V1" gate="G$1" pin="+3V3"/>
-<pinref part="U$1" gate="G$1" pin="VDD"/>
+<pinref part="IC3.01" gate="G$1" pin="VDD"/>
 <wire x1="96.52" y1="147.32" x2="96.52" y2="142.24" width="0.1524" layer="91"/>
 <wire x1="96.52" y1="142.24" x2="104.14" y2="142.24" width="0.1524" layer="91"/>
-<pinref part="U$1" gate="G$1" pin="VDDIO"/>
+<pinref part="IC3.01" gate="G$1" pin="VDDIO"/>
 <wire x1="96.52" y1="142.24" x2="96.52" y2="137.16" width="0.1524" layer="91"/>
 <wire x1="96.52" y1="137.16" x2="104.14" y2="137.16" width="0.1524" layer="91"/>
@@
 <net name="GND" class="0">
 <segment>
-<pinref part="U$1" gate="G$1" pin="GND"/>
+<pinref part="IC3.01" gate="G$1" pin="GND"/>
 <wire x1="104.14" y1="86.36" x2="96.52" y2="86.36" width="0.1524" layer="91"/>
 <pinref part="GND17" gate="1" pin="GND"/>
 <wire x1="96.52" y1="86.36" x2="96.52" y2="81.28" width="0.1524" layer="91"/>
-<pinref part="U$1" gate="G$1" pin="RES"/>
+<pinref part="IC3.01" gate="G$1" pin="RES"/>
 <wire x1="104.14" y1="93.98" x2="96.52" y2="93.98" width="0.1524" layer="91"/>
 <wire x1="96.52" y1="93.98" x2="96.52" y2="86.36" width="0.1524" layer="91"/>
@@
 <net name="N$17" class="0">
 <segment>
-<pinref part="U$1" gate="G$1" pin="DEN_A/G"/>
+<pinref part="IC3.01" gate="G$1" pin="DEN_A/G"/>
 <pinref part="R3.02" gate="G$1" pin="2"/>
 <wire x1="149.86" y1="137.16" x2="200.66" y2="137.16" width="0.1524" layer="91"/>
@@
 <pinref part="R3.04" gate="G$1" pin="2"/>
 <wire x1="213.36" y1="142.24" x2="213.36" y2="132.08" width="0.1524" layer="91"/>
-<pinref part="U$1" gate="G$1" pin="SDO_A/G"/>
+<pinref part="IC3.01" gate="G$1" pin="SDO_A/G"/>
 <wire x1="213.36" y1="132.08" x2="213.36" y2="121.92" width="0.1524" layer="91"/>
 <wire x1="149.86" y1="121.92" x2="193.04" y2="121.92" width="0.1524" layer="91"/>
@@
 <net name="N$26" class="0">
 <segment>
-<pinref part="U$1" gate="G$1" pin="SDO_M"/>
+<pinref part="IC3.01" gate="G$1" pin="SDO_M"/>
 <wire x1="149.86" y1="116.84" x2="195.58" y2="116.84" width="0.1524" layer="91"/>
 <wire x1="195.58" y1="116.84" x2="195.58" y2="129.54" width="0.1524" layer="91"/>
@@
 <segment>
 <pinref part="R3.07" gate="G$1" pin="1"/>
-<pinref part="U$1" gate="G$1" pin="CS_A/G"/>
+<pinref part="IC3.01" gate="G$1" pin="CS_A/G"/>
 <wire x1="177.8" y1="142.24" x2="177.8" y2="111.76" width="0.1524" layer="91"/>
 <wire x1="177.8" y1="111.76" x2="149.86" y2="111.76" width="0.1524" layer="91"/>
@@
 <segment>
 <pinref part="R3.08" gate="G$1" pin="1"/>
-<pinref part="U$1" gate="G$1" pin="CS_M"/>
+<pinref part="IC3.01" gate="G$1" pin="CS_M"/>
 <wire x1="187.96" y1="142.24" x2="187.96" y2="106.68" width="0.1524" layer="91"/>
 <wire x1="187.96" y1="106.68" x2="149.86" y2="106.68" width="0.1524" layer="91"/>
@@
 <net name="!IRQ_GYRO" class="0">
 <segment>
-<pinref part="U$1" gate="G$1" pin="INT1_A/G"/>
+<pinref part="IC3.01" gate="G$1" pin="INT1_A/G"/>
 <wire x1="154.94" y1="86.36" x2="149.86" y2="86.36" width="0.1524" layer="91"/>
 <label x="154.94" y="86.36" size="1.27" layer="95" xref="yes"/>
@@
 <net name="N$1" class="0">
 <segment>
-<pinref part="U$1" gate="G$1" pin="CAP"/>
+<pinref part="IC3.01" gate="G$1" pin="CAP"/>
 <pinref part="C3.01" gate="G$1" pin="1"/>
 <wire x1="104.14" y1="119.38" x2="73.66" y2="119.38" width="0.1524" layer="91"/>
@@
 <segment>
 <pinref part="C3.02" gate="G$1" pin="1"/>
-<pinref part="U$1" gate="G$1" pin="C1"/>
+<pinref part="IC3.01" gate="G$1" pin="C1"/>
 <wire x1="86.36" y1="106.68" x2="86.36" y2="109.22" width="0.1524" layer="91"/>
 <wire x1="86.36" y1="109.22" x2="104.14" y2="109.22" width="0.1524" layer="91"/>

Commit message: Alternative 5V Power Supply added (mb_01.sch)
Parts:
- added C6.01: 100n, rcl:C-EUC0402
- added C6.02: 10u, rcl:C-EUC0603
- added C6.03: 2.2uF, rcl:C-EUC0603
- added C6.04, C6.05: 100u, kitt.psvs:CPOL-29172312
- added FB6.01: BEAD, inductors:BLM15HB121SN1
- added L6.01: NRS8030XX, kitt.psvs:NRS8030XX
- added R6.01: 90k9, rcl:R-EU_R0402
- added R6.02, R6.04, R6.05: 100k, rcl:R-EU_R0402
- added R6.03: 0R02, rcl:R-EU_R0805
- added U1: TPS61032RSARPSDO-G16, kitt.ic:TPS61032RSARPSDO-G16
Connections:
- new net LBO: CON1G$1.ADC.0, R6.04.1, U1.LBO
- new net N$36: FB6.01.2, R6.03.2
- new net N$37: R6.05.1, U1.EN
- new net N$39: L6.01.2, U1.SW, U1.SW_2
- new net N$40: R6.01.2, U1.LBI
- new net N$41: R6.02.2, U1.SYNC
- new net N$43: C6.03.1, C6.04.+, C6.05.+, FB6.01.1, U1.VOUT, U1.VOUT_2, U1.VOUT_3
- net +3V3: now also R6.04.2
- net +4.1V: now also C6.01.1, C6.02.1, L6.01.1, R6.02.1, R6.05.2, U1.VBAT
- net +5V: now also R6.03.1
- net GND: now also C6.01.2, C6.03.2, C6.04.-, C6.05.-, R6.01.1, U1.EP, U1.GND, U1.PGND_3
