File: Hardware/kitt_mb01/eagle/split/mb_01-2.sch (EAGLE design)
At the start: 90 parts, among them CON1 ARDUINO_UNO, IC1.01 RT8293A, IC2.00 BQ24266RGET, IC3.01 LSM9DS1, P1 JST.S2B-PH-SM4-TB, U1 TPS61032RSARPSDO-G16

Commit message: split up project to allow working in parallel
Parts:
- removed C1.01: 22uF/25V, rcl:C-EUC1210K
- removed C1.02, C1.03: 100nF, rcl:C-EUC0402K
- removed C1.04: XX, rcl:C-EUC0402K
- removed C1.05, C1.06: 22uF/6.3V, rcl:C-EUC1206K
- removed C3.01, C3.03, C3.05: 10nF, rcl:C-EUC0402
- removed C3.02: 100nF, rcl:C-EUC0402
- removed C3.04: 10uF, rcl:C-EUC0603K
- removed C4.01: 47uF/25V, rcl:CPOL-EUC/6032-28R
- removed C4.02: 100nF/25V, resistor:C-EUC0603K
- removed C4.03: (no value), resistor:C-EUC0805K
- removed C4.04, C4.05: 220nF/25V, rcl:C-EUC0603K
- removed C6.01: 100n, rcl:C-EUC0402
- removed C6.02: 10u, rcl:C-EUC0603
- removed C6.03: 2.2uF, rcl:C-EUC0603
- removed C6.04, C6.05: 100u, kitt.psvs:CPOL-29172312
- removed CON1: ARDUINO_UNO, kitt.con:ARDUINO_UNO
- removed D1: MBRS320T3, diode:MBRS320T3
- removed F1: 750mA, fuse:MF-SMDF050
- removed FB6.01, L1.01, L2, L4.01: BEAD, inductors:BLM15HB121SN1
- removed IC1: (no value), kitt.ic:DRV8871
- removed IC1.01: RT8293A, kitt.ic:RT8293A
- removed IC3.01: LSM9DS1, kitt.ic:LSM9DS1
- removed L1.02: 4.7uH, rcl:L-EUWE-TPC
- removed L6.01: NRS8030XX, kitt.psvs:NRS8030XX
- removed R1.01: 100kR, rcl:R-EU_R0402
- removed R1.02, R1.03, R1.04: XX, rcl:R-EU_R0402
- removed R1.05, R1.06: [0R], rcl:R-EU_R0402
- removed R2: 10kR, rcl:R-EU_M0805
- removed R3: 2k2R, rcl:R-EU_M0805
- removed R3.01, R3.03: 10kR, rcl:R-EU_R0402
- removed R3.02, R3.04, R3.05, R3.06, R3.07, R3.08: [10kR], rcl:R-EU_R0402
- removed R4.01, R4.02: [0R], rcl:R-EU_M0805
- removed R4.03: 22kR, resistor:R-EU_R0402
- removed R4.04, R4.05: 1kR, resistor:R-EU_R0402
- removed R6.01: 90k9, rcl:R-EU_R0402
- removed R6.02, R6.04, R6.05: 100k, rcl:R-EU_R0402
- removed R6.03: 0R02, rcl:R-EU_R0805
- removed RAILS, SOC, SOC1: (no value), con-phoenix-254:MPT2
- removed REF4: REF_GC-BBV2.0, kitt.con:REF_GC-BBV2.0
- removed REF5: REF.KITT-MB01, kitt.refs:REF.KITT-MB01
- removed SJ1: (no value), jumper:SJ
- removed U1: TPS61032RSARPSDO-G16, kitt.ic:TPS61032RSARPSDO-G16
Connections:
- removed net !IRQ_GYRO: CON1G$3.IO.2, IC3.01.INT1_A/G
- removed net +12V: C4.03.1, D1.C, F1.1, L4.01.2, R2.1
- removed net +3V3: C3.03.1, C3.04.1, C3.05.1, IC3.01.VDD, IC3.01.VDDIO, R3.01.2, R3.03.2, R3.05.2, R3.07.2, R3.08.2, R6.04.2
- removed net GNDA: RAILS-2.1, SJ1.1
- removed net LBO: CON1G$1.ADC.0, R6.04.1, U1.LBO
- removed net MOT.IN1: CON1G$3.IO.3, IC1.IN1, R4.05.2
- removed net MOT.IN2: CON1G$3.IO.4, IC1.IN2, R4.04.2
- removed net N$1: C3.01.1, IC3.01.CAP
- removed net N$10: C4.01.+, C4.02.1, C4.04.1, IC1.VM, L4.01.1
- removed net N$17: IC3.01.DEN_A/G, R3.01.1, R3.02.2
- removed net N$2: F1.2, L1.01.1
- removed net N$23: IC3.01.SDO_A/G, R3.03.1, R3.04.2
- removed net N$24: IC3.01.CS_A/G, R3.07.1
- removed net N$25: C1.04.1, IC1.01.COMP
- removed net N$26: IC3.01.SDO_M, R3.05.1, R3.06.2
- removed net N$27: IC3.01.CS_M, R3.08.1
- removed net N$28: IC1.01.FB, R1.03.1, R1.04.2
- removed net N$29: C1.05.1, C1.06.1, L1.02.1, L2.1, R1.03.2
- removed net N$3: C1.01.1, IC1.01.VIN, L1.01.2, R1.01.1
- removed net N$30: C1.03.2, IC1.01.SW, L1.02.2
- removed net N$31: C1.03.1, IC1.01.BOOT
- removed net N$32: L2.2, R1.05.2, R1.06.1
- removed net N$33: C4.04.2, C4.05.1, IC1.OUT1, SOC1-1.1
- removed net N$34: IC1.OUT2, R4.02.2
- removed net N$35: IC1.ILIM, R4.03.2
- removed net N$36: FB6.01.2, R6.03.2
- removed net N$37: R6.05.1, U1.EN
- removed net N$39: L6.01.2, U1.SW, U1.SW_2
- removed net N$4: IC1.01.EN, R1.01.2
- removed net N$40: R6.01.2, U1.LBI
- removed net N$41: R6.02.2, U1.SYNC
- removed net N$43: C6.03.1, C6.04.+, C6.05.+, FB6.01.1, U1.VOUT, U1.VOUT_2, U1.VOUT_3
- removed net N$5: C1.02.1, IC1.01.SS
- removed net N$6: C3.02.1, IC3.01.C1
- removed net N$7: C1.04.2, R1.02.2
- removed net N$9: R4.01.2, R4.02.1, SOC1-2.1
- removed net RAILS.RX: CON1G$3.IO.0, R2.2, R3.1
- removed net SCL: CON1G$4.SCL
- removed net SDA: CON1G$4.SDA
- removed net VCC/2: D1.A, RAILS-1.1
- net +4.1V: no longer C6.01.1, C6.02.1, L6.01.1, R6.02.1, R6.05.2, U1.VBAT
- net +5V: no longer R1.05.1, R1.06.2, R6.03.1, SOC-1.1
- net GND: no longer C1.01.2, C1.02.2, C1.05.2, C1.06.2, C3.01.2, C3.02.2, C3.03.2, C3.04.2, C3.05.2, C4.01.-, C4.02.2, C4.03.2, C4.05.2, C6.01.2, C6.03.2, C6.04.-, C6.05.-, CON1G$2.GND@1, CON1G$2.GND@2, IC1.01.GND, IC1.01.PAD, IC1.GND, IC1.PAD, IC1.PGND, IC3.01.GND, IC3.01.RES, R1.02.1, R1.04.1, R3.02.1, R3.04.1, R3.06.1, R3.2, R4.01.1, R4.03.1, R4.04.1, R4.05.1, R6.01.1, SJ1.2, SOC-2.1, U1.EP, U1.GND, U1.PGND_3
Other:
- note removed: "- SUPPLY"
- note removed: "D. Hoeglinger"
- note removed: "D.Hoeglinger"
- note removed: "KITT MB01"
- note removed: "KITT MB01 - Axis Sensor"
- note removed: "KITT MB01 - Connectors"
- note removed: "Kit for Intelligent and Trainable Trackcars"
- note removed: "MotorBoard 01"
- note removed: "R01"
