File: Hardware/kitt_mb01/eagle/split/mb_01-4.brd (EAGLE design)
At the start: 160 x 100 mm, 13 parts

Commit message: board parts 4/5 routed
Parts:
- removed R4.01, R4.02: [0R], rcl:M0805
- added SJ1: (no value), jumper:SJ_2
- added U$1: (no value), kitt.refs:REF_GCB2_TS
- moved R4.05 242.7 mm to (67.0, 31.4), turned to 180 degrees
- moved R4.04 237.0 mm to (64.5, 31.4)
- moved R4.03 233.9 mm to (68.9, 30.8), turned to 90 degrees
- moved C4.05 222.6 mm to (67.0, 43.2)
- moved C4.04 218.4 mm to (67.0, 41.6), turned to 180 degrees
- moved L4.01 216.9 mm to (72.4, 41.3)
- moved C4.03 215.3 mm to (72.4, 43.2), turned to 180 degrees
- moved C4.02 208.4 mm to (69.5, 41.3), turned to 90 degrees
- moved C4.01 198.2 mm to (71.8, 35.2), turned to 90 degrees
- moved IC1 181.0 mm to (65.7, 36.5), turned to 90 degrees
- moved SOC1 178.3 mm to (53.7, 28.3), turned to 270 degrees
Connections:
- net GND: now also IC1.7, SJ1.1; no longer IC1.6, R4.01.1
- net N$10: now also IC1.5; no longer IC1.8
- net N$33: now also IC1.6; no longer IC1.7
- net N$34: now also IC1.8, SJ1.3; no longer IC1.5, R4.02.2
- net N$9: now also SJ1.2; no longer R4.01.2, R4.02.1
Routing:
- net N$33: track 0.00 -> 28.9 mm
- net N$34: track 0.00 -> 14.0 mm
- net N$10: track 0.00 -> 9.88 mm
- net N$9: track 0.00 -> 6.99 mm
- net N$35: track 0.00 -> 3.48 mm
- net +12V: track 0.00 -> 2.25 mm
- net MOT.IN2: track 0.00 -> 2.24 mm
- net MOT.IN1: track 0.00 -> 2.24 mm
