File: Hardware/kitt_mb01/eagle/split/mb_01-4.sch (EAGLE design)
At the start: 90 parts, among them CON1 ARDUINO_UNO, IC1.01 RT8293A, IC2.00 BQ24266RGET, IC3.01 LSM9DS1, P1 JST.S2B-PH-SM4-TB, U1 TPS61032RSARPSDO-G16

Commit message: split up project to allow working in parallel
Parts:
- removed C1.01: 22uF/25V, rcl:C-EUC1210K
- removed C1.02, C1.03: 100nF, rcl:C-EUC0402K
- removed C1.04: XX, rcl:C-EUC0402K
- removed C1.05, C1.06: 22uF/6.3V, rcl:C-EUC1206K
- removed C2.01: 1uF/16V, rcl:C-EUC0805
- removed C2.02: 2.2uF/10V, rcl:C-EUC0603K
- removed C2.03: 33nF/16V, rcl:C-EUC0603
- removed C2.04: 33nF/16V, rcl:C-EUC0805
- removed C2.05: 22uF, rcl:CPOL-EUA/3216-18R
- removed C3.01, C3.03, C3.05: 10nF, rcl:C-EUC0402
- removed C3.02: 100nF, rcl:C-EUC0402
- removed C3.04: 10uF, rcl:C-EUC0603K
- removed C6.01: 100n, rcl:C-EUC0402
- removed C6.02: 10u, rcl:C-EUC0603
- removed C6.03: 2.2uF, rcl:C-EUC0603
- removed C6.04, C6.05: 100u, kitt.psvs:CPOL-29172312
- removed CON1: ARDUINO_UNO, kitt.con:ARDUINO_UNO
- removed D1: MBRS320T3, diode:MBRS320T3
- removed F1: 750mA, fuse:MF-SMDF050
- removed FB6.01, L1.01, L2: BEAD, inductors:BLM15HB121SN1
- removed IC1.01: RT8293A, kitt.ic:RT8293A
- removed IC2.00: BQ24266RGET, kitt.ic:BQ24266RGET
- removed IC3.01: LSM9DS1, kitt.ic:LSM9DS1
- removed L1.02: 4.7uH, rcl:L-EUWE-TPC
- removed L2.01: 2.6uH, rcl:L-EUWE-TPC
- removed L2.02: BEAD, rcl:L-EUL2012C
- removed L6.01: NRS8030XX, kitt.psvs:NRS8030XX
- removed P1: JST.S2B-PH-SM4-TB, kitt.con:JST.S2B-PH-SM4-TB
- removed Q1: (no value), transistor-power:P-MOSFET-SO8
- removed R1.01: 100kR, rcl:R-EU_R0402
- removed R1.02, R1.03, R1.04: XX, rcl:R-EU_R0402
- removed R1.05, R1.06: [0R], rcl:R-EU_R0402
- removed R2: 10kR, rcl:R-EU_M0805
- removed R2.01, R2.10, R2.11, R2.12, R2.13, R2.14, R2.15, R3.01, R3.03: 10kR, rcl:R-EU_R0402
- removed R2.02: 31k6R, rcl:R-EU_R0402
- removed R2.03: 1k62R, rcl:R-EU_R0402
- removed R2.04: 5k62R, rcl:R-EU_R0402
- removed R2.05: 11k8R, rcl:R-EU_R0402
- removed R2.06: 10kR/NTC, ptc-ntc:V642
- removed R2.07: 0R, rcl:R-EU_R0402
- removed R2.08: [10kR/NTC], rcl:R-EU_R0402
- removed R3: 2k2R, rcl:R-EU_M0805
- removed R3.02, R3.04, R3.05, R3.06, R3.07, R3.08: [10kR], rcl:R-EU_R0402
- removed R6.01: 90k9, rcl:R-EU_R0402
- removed R6.02, R6.04, R6.05: 100k, rcl:R-EU_R0402
- removed R6.03: 0R02, rcl:R-EU_R0805
- removed RAILS, SOC: (no value), con-phoenix-254:MPT2
- removed REF4: REF_GC-BBV2.0, kitt.con:REF_GC-BBV2.0
- removed REF5: REF.KITT-MB01, kitt.refs:REF.KITT-MB01
- removed SJ1: (no value), jumper:SJ
- removed U1: TPS61032RSARPSDO-G16, kitt.ic:TPS61032RSARPSDO-G16
Connections:
- removed net !IRQ_GYRO: CON1G$3.IO.2, IC3.01.INT1_A/G
- removed net +3V3: C3.03.1, C3.04.1, C3.05.1, IC3.01.VDD, IC3.01.VDDIO, R3.01.2, R3.03.2, R3.05.2, R3.07.2, R3.08.2, R6.04.2
- removed net +4.1V: C2.05.+, C6.01.1, C6.02.1, IC2.00PINS.BAT@1, IC2.00PINS.BAT@2, L6.01.1, P1.1, Q1.D, R2.07.1, R2.10.2, R2.12.2, R2.14.2, R6.02.1, R6.05.2, U1.VBAT
- removed net +5V: IC2.00PINS.IN@1, IC2.00PINS.IN@2, R1.05.1, R1.06.2, R2.02.2, R6.03.1, SOC-1.1
- removed net GNDA: RAILS-2.1, SJ1.1
- removed net IC2.0.!CHG: IC2.00PINS.!CHG
- removed net IC2.0.!PG: IC2.00PINS.!PG
- removed net LBO: CON1G$1.ADC.0, R6.04.1, U1.LBO
- removed net N$1: C3.01.1, IC3.01.CAP
- removed net N$11: IC2.00PINS.VDPM, R2.01.2, R2.02.1
- removed net N$12: C2.03.1, IC2.00PINS.SW@1, IC2.00PINS.SW@2, L2.01.2
- removed net N$13: C2.03.2, IC2.00PINS.BOOT
- removed net N$14: IC2.00PINS.BGATE, Q1.G
- removed net N$15: IC2.00PINS.TS, R2.04.2, R2.05.1, R2.06.2, R2.08.1
- removed net N$16: L2.02.2, R2.07.2
- removed net N$17: IC3.01.DEN_A/G, R3.01.1, R3.02.2
- removed net N$18: C2.04.1, IC2.00PINS.SYS@1, IC2.00PINS.SYS@2, L2.01.1, L2.02.1, Q1.S
- removed net N$19: IC2.00PINS.ISET, R2.03.2
- removed net N$2: F1.2, L1.01.1
- removed net N$20: IC2.00PINS.IUSB@1, R2.10.1, R2.11.2
- removed net N$21: IC2.00PINS.IUSB@2, R2.12.1, R2.13.2
- removed net N$22: IC2.00PINS.IUSB@3, R2.14.1, R2.15.2
- removed net N$23: IC3.01.SDO_A/G, R3.03.1, R3.04.2
- removed net N$24: IC3.01.CS_A/G, R3.07.1
- removed net N$25: C1.04.1, IC1.01.COMP
- removed net N$26: IC3.01.SDO_M, R3.05.1, R3.06.2
- removed net N$27: IC3.01.CS_M, R3.08.1
- removed net N$28: IC1.01.FB, R1.03.1, R1.04.2
- removed net N$29: C1.05.1, C1.06.1, L1.02.1, L2.1, R1.03.2
- removed net N$3: C1.01.1, IC1.01.VIN, L1.01.2, R1.01.1
- removed net N$30: C1.03.2, IC1.01.SW, L1.02.2
- removed net N$31: C1.03.1, IC1.01.BOOT
- removed net N$32: L2.2, R1.05.2, R1.06.1
- removed net N$36: FB6.01.2, R6.03.2
- removed net N$37: R6.05.1, U1.EN
- removed net N$39: L6.01.2, U1.SW, U1.SW_2
- removed net N$4: IC1.01.EN, R1.01.2
- removed net N$40: R6.01.2, U1.LBI
- removed net N$41: R6.02.2, U1.SYNC
- removed net N$43: C6.03.1, C6.04.+, C6.05.+, FB6.01.1, U1.VOUT, U1.VOUT_2, U1.VOUT_3
- removed net N$5: C1.02.1, IC1.01.SS
- removed net N$6: C3.02.1, IC3.01.C1
- removed net N$7: C1.04.2, R1.02.2
- removed net N$8: C2.01.1, IC2.00PINS.PMID
- removed net RAILS.RX: CON1G$3.IO.0, R2.2, R3.1
- removed net SCL: CON1G$4.SCL
- removed net SDA: CON1G$4.SDA
- removed net V+: C2.02.1, IC2.00PINS.DRV, R2.04.1
- removed net VCC/2: D1.A, RAILS-1.1
- net +12V: no longer D1.C, F1.1, R2.1
- net GND: no longer C1.01.2, C1.02.2, C1.05.2, C1.06.2, C2.01.2, C2.02.2, C2.04.2, C2.05.-, C3.01.2, C3.02.2, C3.03.2, C3.04.2, C3.05.2, C6.01.2, C6.03.2, C6.04.-, C6.05.-, CON1G$2.GND@1, CON1G$2.GND@2, IC1.01.GND, IC1.01.PAD, IC2.00PAD.THERMAL, IC2.00PINS.AGND, IC2.00PINS.PGND@1, IC2.00PINS.PGND@2, IC3.01.GND, IC3.01.RES, P1.2, R1.02.1, R1.04.1, R2.01.1, R2.03.1, R2.05.2, R2.06.1, R2.08.2, R2.11.1, R2.13.1, R2.15.1, R3.02.1, R3.04.1, R3.06.1, R3.2, R6.01.1, SJ1.2, SOC-2.1, U1.EP, U1.GND, U1.PGND_3
- net MOT.IN1: no longer CON1G$3.IO.3
- net MOT.IN2: no longer CON1G$3.IO.4
Other:
- note removed: "- SUPPLY"
- note removed: "D. Hoeglinger"
- note removed: "D.Hoeglinger"
- note removed: "KITT MB01"
- note removed: "KITT MB01 - Axis Sensor"
- note removed: "KITT MB01 - Battery Charger"
- note removed: "KITT MB01 - Connectors"
- note removed: "Kit for Intelligent and Trainable Trackcars"
- note removed: "MotorBoard 01"
- note removed: "R01"

Commit message: board parts 4/5 routed
Parts:
- removed R4.01, R4.02: [0R], rcl:R-EU_M0805
- added SJ1: (no value), jumper:SJ2W
Connections:
- net GND: now also SJ1.1; no longer R4.01.1
- net N$34: now also SJ1.3; no longer R4.02.2
- net N$9: now also SJ1.2; no longer R4.01.2, R4.02.1
Other:
- moved on the sheet: SOC1-2
Changed lines of the file:
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@@
 <part name="GND22" library="supply1" deviceset="GND" device=""/>
 <part name="GND23" library="supply1" deviceset="GND" device=""/>
-<part name="R4.01" library="rcl" deviceset="R-EU_" device="M0805" value="[0R]"/>
-<part name="R4.02" library="rcl" deviceset="R-EU_" device="M0805" value="[0R]"/>
 <part name="R4.03" library="resistor" deviceset="R-EU_" device="R0402" value="22kR"/>
 <part name="R4.04" library="resistor" deviceset="R-EU_" device="R0402" value="1kR"/>
 <part name="R4.05" library="resistor" deviceset="R-EU_" device="R0402" value="1kR"/>
+<part name="SJ1" library="jumper" deviceset="SJ2W" device=""/>
 </parts>
 <sheets>
@@
 <instance part="IC1" gate="G$1" x="149.86" y="91.44"/>
 <instance part="SOC1" gate="-1" x="220.98" y="99.06" rot="MR180"/>
-<instance part="SOC1" gate="-2" x="220.98" y="86.36" rot="MR180"/>
+<instance part="SOC1" gate="-2" x="220.98" y="81.28" rot="MR180"/>
 <instance part="C4.01" gate="G$1" x="88.9" y="121.92" rot="MR0"/>
 <instance part="C4.02" gate="G$1" x="68.58" y="121.92" rot="MR0"/>
@@
 <instance part="GND22" gate="1" x="203.2" y="55.88" rot="MR0"/>
 <instance part="GND23" gate="1" x="149.86" y="55.88" rot="MR0"/>
-<instance part="R4.01" gate="G$1" x="193.04" y="73.66" rot="R90"/>
-<instance part="R4.02" gate="G$1" x="182.88" y="86.36" rot="MR0"/>
 <instance part="R4.03" gate="G$1" x="119.38" y="73.66" rot="R90"/>
 <instance part="R4.04" gate="G$1" x="109.22" y="73.66" rot="R90"/>
 <instance part="R4.05" gate="G$1" x="99.06" y="73.66" rot="R90"/>
+<instance part="SJ1" gate="G$1" x="193.04" y="81.28" rot="R180"/>
 </instances>
 <busses>
@@
 <segment>
 <pinref part="SOC1" gate="-2" pin="1"/>
-<wire x1="218.44" y1="86.36" x2="193.04" y2="86.36" width="0.1524" layer="91"/>
-<pinref part="R4.01" gate="G$1" pin="2"/>
-<wire x1="193.04" y1="78.74" x2="193.04" y2="86.36" width="0.1524" layer="91"/>
-<pinref part="R4.02" gate="G$1" pin="1"/>
-<wire x1="187.96" y1="86.36" x2="193.04" y2="86.36" width="0.1524" layer="91"/>
-<junction x="193.04" y="86.36"/>
+<wire x1="218.44" y1="81.28" x2="198.12" y2="81.28" width="0.1524" layer="91"/>
+<pinref part="SJ1" gate="G$1" pin="2"/>
 </segment>
 </net>
@@
 <pinref part="GND22" gate="1" pin="GND"/>
 <wire x1="203.2" y1="68.58" x2="203.2" y2="60.96" width="0.1524" layer="91"/>
-<pinref part="R4.01" gate="G$1" pin="1"/>
 <wire x1="203.2" y1="60.96" x2="203.2" y2="58.42" width="0.1524" layer="91"/>
-<wire x1="193.04" y1="68.58" x2="193.04" y2="60.96" width="0.1524" layer="91"/>
+<wire x1="193.04" y1="76.2" x2="193.04" y2="60.96" width="0.1524" layer="91"/>
 <wire x1="193.04" y1="60.96" x2="203.2" y2="60.96" width="0.1524" layer="91"/>
 <junction x="203.2" y="60.96"/>
+<pinref part="SJ1" gate="G$1" pin="1"/>
 </segment>
 <segment>
@@
 <net name="N$34" class="0">
 <segment>
-<pinref part="R4.02" gate="G$1" pin="2"/>
 <pinref part="IC1" gate="G$1" pin="OUT2"/>
-<wire x1="177.8" y1="86.36" x2="172.72" y2="86.36" width="0.1524" layer="91"/>
+<wire x1="193.04" y1="86.36" x2="172.72" y2="86.36" width="0.1524" layer="91"/>
+<pinref part="SJ1" gate="G$1" pin="3"/>
 </segment>
 </net>
