File: Hardware/kitt_mb01/eagle/split/mb_01-5.brd (EAGLE design)
At the start: 160 x 100 mm, 13 parts, among them U1 TPS61032RSARPSDO-G16

Commit message: board parts 4/5 routed
Parts:
- added U$1: (no value), kitt.refs:REF_GCB2_TS
- added U$2: (no value), kitt.refs:REF_GCB2_BS
- moved L6.01 299.3 mm to (66.4, 40.0), flipped to the bottom
- moved C6.05 293.1 mm to (67.9, 31.8), flipped to the bottom, turned to 90 degrees
- moved C6.02 290.7 mm to (71.8, 37.1), flipped to the bottom, turned to 270 degrees
- moved C6.01 288.2 mm to (75.6, 36.8), flipped to the bottom, turned to 270 degrees
- moved C6.04 288.1 mm to (64.5, 31.8), flipped to the bottom, turned to 90 degrees
- moved R6.03 286.4 mm to (88.6, 51.1), turned to 270 degrees
- moved R6.02 286.3 mm to (80.0, 41.3), flipped to the bottom, turned to 90 degrees
- moved R6.01 283.4 mm to (74.3, 36.8), flipped to the bottom, turned to 270 degrees
- moved FB6.01 282.2 mm to (62.9, 26.7), flipped to the bottom
- moved R6.05 267.0 mm to (75.2, 26.7), flipped to the bottom, turned to 270 degrees
- moved R6.04 262.8 mm to (74.0, 26.7), flipped to the bottom, turned to 270 degrees
- moved C6.03 252.1 mm to (71.8, 27.0), flipped to the bottom, turned to 180 degrees
- moved U1 249.4 mm to (72.7, 31.8), flipped to the bottom, turned to 180 degrees
Connections:
- net GND: now also C6.02.2, U1.3, U1.4
Routing:
- net +4.1V: track 0.00 -> 34.7 mm
- net N$43: track 0.00 -> 16.4 mm
- net N$39: track 0.00 -> 13.2 mm
- net N$41: track 0.00 -> 12.4 mm, vias 0 -> 2
- net LBO: track 0.00 -> 1.88 mm
- net N$37: track 0.00 -> 1.80 mm
- net N$40: track 0.00 -> 1.57 mm
