File: Hardware/kitt_mb01/eagle/split/mb_01-1.sch (EAGLE design)
At the start: 19 parts, among them IC1.01 RT8293A

Commit message: did route+place for subsection 1 and 3
Parts:
- F1: device fuse:MF-SMDF050 -> rcl:R-EU_R0805
- L1.02: device rcl:L-EUWE-TPC -> kitt.psvs:NRS8030XX
Changed lines of the file:
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@@
 <parts>
 <part name="D1" library="diode" deviceset="MBRS3*0T3" device="" technology="2"/>
-<part name="F1" library="fuse" deviceset="MF-SMDF" device="" technology="050" value="750mA"/>
+<part name="F1" library="rcl" deviceset="R-EU_" device="R0805" value="750mA"/>
 <part name="L1.01" library="inductors" deviceset="BLM15H" device="" technology="B121SN1" value="BEAD"/>
 <part name="P+2" library="supply1" deviceset="+12V" device="" value="V.POW"/>
@@
 <part name="C1.01" library="rcl" deviceset="C-EU" device="C1210K" value="22uF/25V"/>
 <part name="GND3" library="supply1" deviceset="GND" device=""/>
-<part name="L1.02" library="rcl" deviceset="L-EU" device="WE-TPC" value="4.7uH"/>
+<part name="L1.02" library="kitt.psvs" deviceset="NRS8030XX" device="" value="4.7uH"/>
 <part name="P+5VMAIN" library="supply1" deviceset="+5V" device="" value="+5V-MAIN"/>
 <part name="L2" library="inductors" deviceset="BLM15H" device="" technology="B121SN1" value="BEAD"/>
@@
 <instances>
 <instance part="D1" gate="G$1" x="31.75" y="151.13"/>
-<instance part="F1" gate="A" x="49.53" y="151.13"/>
+<instance part="F1" gate="G$1" x="49.53" y="151.13"/>
 <instance part="L1.01" gate="G$1" x="62.23" y="151.13"/>
 <instance part="P+2" gate="1" x="41.91" y="158.75" smashed="yes">
@@
 <net name="N$2" class="0">
 <segment>
-<pinref part="F1" gate="A" pin="2"/>
+<pinref part="F1" gate="G$1" pin="2"/>
 <pinref part="L1.01" gate="G$1" pin="1"/>
 <wire x1="54.61" y1="151.13" x2="57.15" y2="151.13" width="0.1524" layer="91"/>
@@
 <segment>
 <pinref part="D1" gate="G$1" pin="C"/>
-<pinref part="F1" gate="A" pin="1"/>
+<pinref part="F1" gate="G$1" pin="1"/>
 <wire x1="34.29" y1="151.13" x2="41.91" y2="151.13" width="0.1524" layer="91"/>
 <pinref part="P+2" gate="1" pin="+12V"/>
