File: Hardware/kitt_mb01/eagle/merge/mb01-merge.brd (EAGLE design)
At the start: 160 x 100 mm, 21 parts, among them IC1.01 RT8293A

Commit message: did route+place for subsection 1 and 3
Parts:
- F1: device rcl:R0805 -> fuse:MF-SMDF050
- L1.02: device kitt.psvs:TAIYO-YUDEN.NRS8030T4R7MJGJ -> rcl:POWER-CHOKE_WE-TPC
- moved R1.06 324.2 mm to (-25.4, -223.5)
- moved R1.05 318.1 mm to (-25.4, -218.4), turned to 0 degrees
- moved D1 139.4 mm to (126.1, -64.0)
- moved C1.03 133.8 mm to (47.6, -53.0)
- moved F1 131.9 mm to (126.3, -55.2), turned to 90 degrees
- moved L2 123.5 mm to (38.1, -28.9)
- moved C1.05 121.1 mm to (51.1, -39.1), turned to 90 degrees
- moved R1.04 120.7 mm to (39.7, -44.1)
- moved R1.02 120.5 mm to (42.9, -44.5)
- moved C1.01 120.5 mm to (40.4, -32.8)
- moved C1.02 120.2 mm to (45.1, -44.8)
- moved IC1.01 120.2 mm to (41.3, -38.4)
- moved C1.04 119.7 mm to (41.6, -43.8)
- moved R1.01 119.7 mm to (45.1, -38.1)
- moved R1.03 118.3 mm to (39.7, -42.9)
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Routing:
- net N$29: track 27.4 -> 0.00 mm
- net GND: track 20.5 -> 0.00 mm, vias 1 -> 0
- net N$30: track 16.2 -> 0.00 mm, vias 9 -> 0
- net N$3: track 10.8 -> 0.00 mm
- net +12V: track 5.00 -> 0.00 mm
- net N$2: track 2.23 -> 0.00 mm
- net N$31: track 1.73 -> 0.00 mm
- net N$7: track 2.72 -> 1.41 mm
- net N$5: track 3.06 -> 4.09 mm
- net N$28: track 4.23 -> 3.36 mm
- net N$4: track 6.40 -> 6.95 mm
- removed copper zone on layer 2, net N$30
Other:
- board size 160 x 100 mm -> 160 x 204.1 mm
