File: Hardware/kitt_db01/eagle/kitt_db01.sch (EAGLE design)
At the start: 101 parts, among them U9.00 ADNS-3080, U9.01 MIC5205-3.3YM5TR, U9.02 SI1922EDH, X9.00 RESON

Commit message: snapshot of db01 board layout : so much wasted space edition -> top and botton silk screen names complete -> power plane, ground and stitching done -> some minor route optimization done
Parts:
- added R9.16, R9.17: 10kR, rcl:R-EU_R0805
Connections:
- net GND: now also R9.16.2, R9.17.2
- net N$184: now also R9.16.1
- net N$4: now also R9.17.1
Changed lines of the file:
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@@
 <setting verticaltext="up"/>
 </settings>
-<grid distance="0.1" unitdist="inch" unit="inch" style="lines" multiple="1" display="no" altdistance="0.01" altunitdist="inch" altunit="inch"/>
+<grid distance="0.05" unitdist="inch" unit="inch" style="lines" multiple="1" display="no" altdistance="0.01" altunitdist="inch" altunit="inch"/>
 <layers>
 <layer number="1" name="Top" color="4" fill="1" visible="no" active="no"/>
@@
 <part name="+3V10" library="supply1" deviceset="+3V3" device=""/>
 <part name="P+3" library="supply1" deviceset="+5V" device=""/>
+<part name="R9.16" library="rcl" deviceset="R-EU_" device="R0805" value="10kR"/>
+<part name="GND13" library="supply1" deviceset="GND" device=""/>
+<part name="R9.17" library="rcl" deviceset="R-EU_" device="R0805" value="10kR"/>
+<part name="GND14" library="supply1" deviceset="GND" device=""/>
 </parts>
 <sheets>
@@
 <instance part="+3V10" gate="G$1" x="87.63" y="72.39"/>
 <instance part="P+3" gate="1" x="97.79" y="72.39" rot="MR0"/>
+<instance part="R9.16" gate="G$1" x="217.17" y="54.61" rot="MR270"/>
+<instance part="GND13" gate="1" x="217.17" y="44.45"/>
+<instance part="R9.17" gate="G$1" x="180.34" y="54.61" rot="MR270"/>
+<instance part="GND14" gate="1" x="180.34" y="44.45"/>
 </instances>
 <busses>
@@
 <wire x1="85.09" y1="39.37" x2="85.09" y2="43.18" width="0.1524" layer="91"/>
 </segment>
+<segment>
+<pinref part="R9.16" gate="G$1" pin="2"/>
+<pinref part="GND13" gate="1" pin="GND"/>
+<wire x1="217.17" y1="46.99" x2="217.17" y2="49.53" width="0.1524" layer="91"/>
+</segment>
+<segment>
+<pinref part="R9.17" gate="G$1" pin="2"/>
+<pinref part="GND14" gate="1" pin="GND"/>
+<wire x1="180.34" y1="46.99" x2="180.34" y2="49.53" width="0.1524" layer="91"/>
+</segment>
 </net>
 <net name="MOSI" class="0">
@@
 <wire x1="180.34" y1="76.2" x2="180.34" y2="85.09" width="0.1524" layer="91"/>
 <pinref part="U9.02" gate="A" pin="G"/>
+<pinref part="R9.17" gate="G$1" pin="1"/>
+<wire x1="180.34" y1="59.69" x2="180.34" y2="76.2" width="0.1524" layer="91"/>
+<junction x="180.34" y="76.2"/>
 </segment>
 </net>
@@
 <wire x1="217.17" y1="66.04" x2="217.17" y2="76.2" width="0.1524" layer="91"/>
 <junction x="217.17" y="76.2"/>
-</segment>
-</net>
+<pinref part="R9.16" gate="G$1" pin="1"/>
+<wire x1="217.17" y1="59.69" x2="217.17" y2="66.04" width="0.1524" layer="91"/>
+<junction x="217.17" y="66.04"/>
+</segment>
+</net>

Commit message: added logos, text and decals on bottom side
Parts:
- added DCL1: DCL.CARRERAI, kitt.refs:DCL.CARRERAI
- added DCL2: DCL.OSH.COPPER'5MM', kitt.refs:DCL.OSH.COPPER'5MM'
- added REF1: REF.LOGO.UASUA, kitt.refs:REF.LOGO.UASUA
Changed lines of the file:
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@@
 <setting verticaltext="up"/>
 </settings>
-<grid distance="0.05" unitdist="inch" unit="inch" style="lines" multiple="1" display="no" altdistance="0.01" altunitdist="inch" altunit="inch"/>
+<grid distance="0.1" unitdist="inch" unit="inch" style="lines" multiple="1" display="no" altdistance="0.01" altunitdist="inch" altunit="inch"/>
 <layers>
 <layer number="1" name="Top" color="4" fill="1" visible="no" active="no"/>
@@
 <part name="R9.17" library="rcl" deviceset="R-EU_" device="R0805" value="10kR"/>
 <part name="GND14" library="supply1" deviceset="GND" device=""/>
+<part name="DCL1" library="kitt.refs" deviceset="DCL.CARRERAI" device=""/>
+<part name="REF1" library="kitt.refs" deviceset="REF.LOGO.UASUA" device=""/>
+<part name="DCL2" library="kitt.refs" deviceset="DCL.OSH.COPPER" device="'5MM'"/>
 </parts>
 <sheets>
@@
 <instance part="R9.17" gate="G$1" x="180.34" y="54.61" rot="MR270"/>
 <instance part="GND14" gate="1" x="180.34" y="44.45"/>
+<instance part="DCL1" gate="G$1" x="162.56" y="27.94"/>
+<instance part="REF1" gate="G$1" x="162.56" y="33.02"/>
+<instance part="DCL2" gate="G$1" x="185.42" y="27.94"/>
 </instances>
 <busses>
