File: Hardware/baseboard/eagle/main.sch (EAGLE design)
At the start: 84 parts, among them P1 JST.S2B-PH-SM4-TB, Q5.XX2 PCF/XX, Q5.XX3 PCF/XX, U3.1 LSM9DS1, U4 TPS61032RSARP˸^)SDO-G16, U5 LTC4000-1, X1.0 ARDUINO_UNO, X1.2 TACH/LAP, X2.1 MOTOR, X2.2 MOTOR

Commit message: tried out EAGLEv7's module feature , looks promising
Parts:
- removed C5.XX2: 1uF/XX, rcl:C-EU025-024X044
- removed C5.XX3, C5.XX4: 10nF/XX, rcl:C-EU025-024X044
- removed C5.XX5, C5.XX6: F/XX, rcl:C-EU025-024X044
- removed Q5.XX2, Q5.XX3: PCF/XX, transistor-power:IRF4905
- removed R5.XX10: 82kR/XX, rcl:R-EU_0204/5
- removed R5.XX11, R5.XX4, R5.XX5: 100kR/XX, rcl:R-EU_0204/5
- removed R5.XX12: 270kR/XX, rcl:R-EU_0204/5
- removed R5.XX13: 5mR/XX, rcl:R-EU_0204/5
- removed R5.XX2, R5.XX3: 1kR/XX, rcl:R-EU_0204/5
- removed R5.XX6: 0.82R/XX, rcl:R-EU_0204/5
- removed R5.XX7: 16kR/XX, rcl:R-EU_0204/5
- removed R5.XX8: 1MR/XX, rcl:R-EU_0204/5
- removed R5.XX9: 220kR/XX, rcl:R-EU_0204/5
- removed U5: LTC4000-1, kitt.ic:LTC4000-1
- removed ☇5XX2, ☇5XX3, ☇5XX4, ☇5XX5, ☇5XX6, ☇5XX7, ☇5XX8, ☇5XX9: PTR1TP07SQ, testpad:PTR1TP07SQ
Connections:
- removed net BAT.+: Q5.XX3.D, R5.XX9.2, U5.BAT
- removed net BAT.NTC: U5.NTC
- removed net DDC.!RST: U5.!RST
- removed net DDC.IN: Q5.XX2.S, R5.XX6.2, U5.CLN, U5.IID, ☇5XX6.TP
- removed net N$13: R5.XX2.2, U5.CX
- removed net N$15: R5.XX4.1, U5.!CHRG
- removed net N$16: R5.XX5.1, U5.!FLT
- removed net N$19: C5.XX5.1, R5.XX7.1
- removed net N$20: C5.XX5.2, U5.CC
- removed net N$21: R5.XX7.2, U5.ITH
- removed net N$23: Q5.XX2.G, R5.XX8.2, U5.IGATE
- removed net N$24: R5.XX10.1, R5.XX9.1, U5.BFB
- removed net N$26: R5.XX11.2, R5.XX12.1, U5.OFB
- removed net N$27: Q5.XX3.S, R5.XX13.1, U5.CSN
- removed net N$28: Q5.XX3.G, U5.BGATE
- removed net N5.BIAS: C5.XX2.1, R5.XX4.2, R5.XX5.2, U5.BIAS, U5.VM
- removed net N5.CL: R5.XX3.2, U5.CL, ☇5XX9.TP
- removed net N5.ENC: U5.ENC, ☇5XX3.TP
- removed net N5.FBG: R5.XX10.2, R5.XX11.1, U5.FBG, ☇5XX5.TP
- removed net N5.IBMON: C5.XX4.1, U5.IBMON, ☇5XX7.TP
- removed net N5.IFB: U5.IFB, ☇5XX4.TP
- removed net N5.IIMON: C5.XX3.1, U5.IIMON, ☇5XX8.TP
- removed net N5.TMR: U5.TMR, ☇5XX2.TP
- net GND: no longer C5.XX2.2, C5.XX3.2, C5.XX4.2, C5.XX6.2, R5.XX2.1, R5.XX3.1, U5.GND
- net VCC/2: no longer C5.XX6.1, Q5.XX2.D, R5.XX12.2, R5.XX13.2, R5.XX6.1, R5.XX8.1, U5.CSP, U5.IN

Commit message: quicksave ; before adding in DC/DC input component
Other:
- note added: "✔"
Changed lines of the file:
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@@
 </text>
 <text x="43.18" y="15.24" size="1.778" layer="98">(TURN OFF)</text>
+<text x="40.64" y="-10.16" size="5.08" layer="98">✔</text>
 </plain>
 <moduleinsts>
-<moduleinst name="A5-U1" module="POW-4001" x="76.2" y="76.2" smashed="yes">
-<attribute name="NAME" x="76.2" y="71.12" size="2.032" layer="95" align="bottom-center"/>
+<moduleinst name="A5-U1" module="POW-4001" x="86.36" y="63.5" smashed="yes">
+<attribute name="NAME" x="86.36" y="58.42" size="2.032" layer="95" align="bottom-center"/>
 </moduleinst>
 </moduleinsts>
@@
 [ ] Schematic/Peer Review</text>
 <text x="124.46" y="55.88" size="1.778" layer="98">PfaffM(sic): No point in making separate GND zones, focus on preventing slit antennae</text>
+<text x="1.27" y="-5.08" size="1.778" layer="98">✔</text>
 </plain>
 <instances>
@@
 [  ] Name nets on pins after pins connected for routing later,
      maybe use some unicode symbol for proximity constraints?</text>
+<text x="0" y="-25.4" size="6.4516" layer="98">✔</text>
 </plain>
 <instances>

Commit message: entered LTC3891 into schematic ; also added a liberal amount of testpoints , for both control signals , and DC/DC measurements
Other:
- note added: "COMPONENT MASTERS"

Commit message: quicksave ; rearranged the module ports of A5 and A6 , this looks amazing so far
Changed lines of the file:
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@@
 <module name="POW-4001" prefix="A5" dx="45.72" dy="30.48">
 <ports>
-<port name="DDC.IN" side="top" coord="-12.7" direction="io"/>
-<port name="DDC.OUT" side="top" coord="12.7" direction="io"/>
-<port name="DDC.!RST" side="top" coord="0" direction="out"/>
+<port name="DDC.IN" side="top" coord="-5.08" direction="io"/>
+<port name="DDC.OUT" side="top" coord="10.16" direction="io"/>
+<port name="DDC.!RST" side="left" coord="2.54" direction="out"/>
 <port name="BAT.+" side="right" coord="-5.08" direction="pwr"/>
 <port name="BAT.NTC" side="right" coord="-10.16" direction="in"/>
-<port name="GND" side="bottom" coord="0" direction="pwr"/>
-<port name="VDD" side="left" coord="2.54" direction="pwr"/>
+<port name="GND" side="left" coord="-10.16" direction="pwr"/>
+<port name="VDD" side="left" coord="10.16" direction="pwr"/>
 <port name="VSYS" side="right" coord="2.54" direction="pwr"/>
+<port name="DDC.ITH" side="top" coord="2.54" direction="io"/>
 </ports>
 <variantdefs>
@@
 </sheets>
 </module>
-<module name="POW-3891" prefix="A6" dx="45.72" dy="30.48">
+<module name="POW-3891" prefix="A6" dx="45.72" dy="35.56">
 <ports>
+<port name="DDC.VIN" side="bottom" coord="-5.08" direction="io"/>
+<port name="DDC.ITH" side="bottom" coord="2.54" direction="io"/>
+<port name="DDC.OUT" side="bottom" coord="10.16" direction="io"/>
+<port name="CTRL.RUN" side="left" coord="12.7" direction="in"/>
+<port name="CTRL.PGOOD" side="left" coord="7.62" direction="out"/>
+<port name="CTRL.PLLIN/MODE" side="left" coord="2.54" direction="in"/>
+<port name="CTRL.FREQ" side="left" coord="-2.54" direction="in"/>
+<port name="GND" side="left" coord="-12.7" direction="pwr"/>
+<port name="DDC.EXTVCC" side="right" coord="12.7" direction="pwr"/>
 </ports>
 <variantdefs>
@@
 <net name="N6.EXTVCC" class="0">
 <segment>
+<wire x1="129.54" y1="22.86" x2="144.78" y2="22.86" width="0.1524" layer="91"/>
+<pinref part="☇6XX1" gate="G$1" pin="TP"/>
+<label x="144.78" y="25.4" size="1.778" layer="95" rot="R180"/>
+</segment>
+</net>
+<net name="DDC.EXTVCC" class="0">
+<segment>
 <pinref part="U6" gate="A" pin="EXTVCC"/>
 <wire x1="116.84" y1="139.7" x2="132.08" y2="139.7" width="0.1524" layer="91"/>
 <label x="132.08" y="142.24" size="1.778" layer="95" rot="R180"/>
-</segment>
-<segment>
-<wire x1="129.54" y1="22.86" x2="144.78" y2="22.86" width="0.1524" layer="91"/>
-<pinref part="☇6XX1" gate="G$1" pin="TP"/>
-<label x="144.78" y="25.4" size="1.778" layer="95" rot="R180"/>
 </segment>
 </net>
@@
 <part name="P+8" library="supply1" deviceset="VCC/2" device="" value="SYSV"/>
 <part name="P1" library="kitt.con" deviceset="JST.S2B-PH-SM4-TB" device=""/>
+<part name="FRAME5" library="frames" deviceset="A4L-LOC" device=""/>
 </parts>
 <sheets>
@@
 <text x="40.64" y="-10.16" size="5.08" layer="98">✔</text>
 </plain>
-<moduleinsts>
-<moduleinst name="A5-U1" module="POW-4001" x="114.3" y="63.5" smashed="yes">
-<attribute name="NAME" x="114.3" y="58.42" size="2.032" layer="95" align="bottom-center"/>
-</moduleinst>
-<moduleinst name="A6-1" module="POW-3891" x="114.3" y="109.22"/>
-</moduleinsts>
 <instances>
 <instance part="FRAME1" gate="G$1" x="0" y="0"/>
@@
 </segment>
 </net>
+</nets>
+</sheet>
+<sheet>
+<description>POW-System Supply Chain</description>
+<plain>
+</plain>
+<moduleinsts>
+<moduleinst name="A5-U1" module="POW-4001" x="111.76" y="73.66" smashed="yes">
+<attribute name="NAME" x="88.9" y="91.44" size="2.032" layer="95"/>
+</moduleinst>
+<moduleinst name="A6-U1" module="POW-3891" x="111.76" y="119.38" smashed="yes">
+<attribute name="NAME" x="88.9" y="139.7" size="2.032" layer="95"/>
+</moduleinst>
+</moduleinsts>
+<instances>
+<instance part="FRAME5" gate="G$1" x="0" y="0"/>
+</instances>
+<busses>
+</busses>
+<nets>
+<net name="N$13" class="0">
+<segment>
+<portref moduleinst="A6-U1" port="DDC.VIN"/>
+<portref moduleinst="A5-U1" port="DDC.IN"/>
+<wire x1="106.68" y1="96.52" x2="106.68" y2="93.98" width="0.1524" layer="91"/>
+</segment>
+</net>
+<net name="N$14" class="0">
+<segment>
+<portref moduleinst="A6-U1" port="DDC.OUT"/>
+<portref moduleinst="A5-U1" port="DDC.OUT"/>
+<wire x1="121.92" y1="96.52" x2="121.92" y2="93.98" width="0.1524" layer="91"/>
+</segment>
+</net>
+<net name="N$15" class="0">
+<segment>
+<portref moduleinst="A6-U1" port="DDC.ITH"/>
+<portref moduleinst="A5-U1" port="DDC.ITH"/>
+<wire x1="114.3" y1="96.52" x2="114.3" y2="93.98" width="0.1524" layer="91"/>
+</segment>
+</net>
