File: Hardware/baseboard/eagle/main.sch (EAGLE design)
At the start: 32 parts, among them X1 JST-4POS-2X4POS, X1.2 TACH/LAP, X2 ATLAS-LTC, X2.1 MOTOR, X2.2 VRAILS+, X2.3 5V+SoC, X3 SYS-IIC, X4 SYSTEWI

Commit message: wip baseboard + as announced, added breakaway LTC connector + threw in molex/wirepad power thing too   because it looks symmetrical and the fab house would like   the board to be rectangular I guess
Parts:
- added X5: 15244441, kitt.con:15244441
- added ⌁1: SINGLEPAD40MIL-BREAK.PILOT, kitt.con:SINGLEPAD40MIL-BREAK.PILOT
- added ⌁2, ⌁3: SINGLEPAD40MIL-BREAK, kitt.con:SINGLEPAD40MIL-BREAK
Connections:
- new net V++: ⌁2.P$1
- net +5V: now also X5.4, ⌁3.P$1
- net GND: now also X5.2, X5.3, ⌁1.P$1, ⌁2.P$1
- net VCC/2: now also X5.1, ⌁1.P$1
- net VSYS: now also ⌁3.P$1
Other:
- note added: "for developers who dislike screwing around with phoenix contact 100mil connectors - breakaway next to LTC connector"
Changed lines of the file:
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@@
 <part name="SUPPLY3" library="supply2" deviceset="+4.1V" device=""/>
 <part name="D1" library="diode" deviceset="BAS40-05" device=""/>
+<part name="X5" library="kitt.con" deviceset="15244441" device=""/>
+<part name="P+9" library="supply1" deviceset="VCC/2" device="" value="VRAILS"/>
+<part name="GND6" library="supply1" deviceset="GND" device=""/>
+<part name="P+10" library="supply1" deviceset="+5V" device=""/>
+<part name="⌁1" library="kitt.con" deviceset="SINGLEPAD" device="40MIL-BREAK.PILOT"/>
+<part name="⌁2" library="kitt.con" deviceset="SINGLEPAD" device="40MIL-BREAK" value="SINGLEPAD40MIL-BREAK"/>
+<part name="⌁3" library="kitt.con" deviceset="SINGLEPAD" device="40MIL-BREAK" value="SINGLEPAD40MIL-BREAK"/>
 </parts>
 <sheets>
@@
 Look at Battery In:
 Capacitor and ESD38, what's this?</text>
+<text x="12.7" y="180.34" size="1.778" layer="98" ratio="20" align="center-left">for developers who dislike screwing around
+with phoenix contact 100mil connectors
+- breakaway next to LTC connector</text>
 </plain>
 <moduleinsts>
@@
 <instance part="X1" gate="B" x="314.96" y="49.53" rot="MR180"/>
 <instance part="SUPPLY2" gate="P" x="264.16" y="83.82"/>
+<instance part="X5" gate="G$1" x="22.86" y="162.56" rot="MR0"/>
+<instance part="P+9" gate="G$1" x="40.64" y="167.64" rot="R270"/>
+<instance part="GND6" gate="1" x="35.56" y="152.4" rot="MR0"/>
+<instance part="P+10" gate="1" x="43.18" y="160.02" smashed="yes" rot="MR90">
+<attribute name="VALUE" x="39.37" y="163.83" size="1.778" layer="96" rot="MR180"/>
+</instance>
+<instance part="⌁1" gate="G$1" x="35.56" y="167.64" rot="R90"/>
+<instance part="⌁2" gate="G$1" x="35.56" y="165.1" rot="R90"/>
+<instance part="⌁3" gate="G$1" x="38.1" y="160.02" rot="R90"/>
 </instances>
 <busses>
@@
 <pinref part="GND4" gate="1" pin="GND"/>
 </segment>
+<segment>
+<pinref part="X5" gate="G$1" pin="2"/>
+<pinref part="GND6" gate="1" pin="GND"/>
+<wire x1="30.48" y1="165.1" x2="35.56" y2="165.1" width="0.1524" layer="91"/>
+<wire x1="35.56" y1="165.1" x2="35.56" y2="162.56" width="0.1524" layer="91"/>
+<pinref part="X5" gate="G$1" pin="3"/>
+<wire x1="35.56" y1="162.56" x2="35.56" y2="154.94" width="0.1524" layer="91"/>
+<wire x1="30.48" y1="162.56" x2="35.56" y2="162.56" width="0.1524" layer="91"/>
+<junction x="35.56" y="162.56"/>
+<pinref part="⌁2" gate="G$1" pin="P$1"/>
+<junction x="35.56" y="165.1"/>
+</segment>
 </net>
 <net name="+18V" class="0">
@@
 <portref moduleinst="A4" port="V~IN"/>
 </segment>
+<segment>
+<pinref part="X5" gate="G$1" pin="1"/>
+<pinref part="P+9" gate="G$1" pin="VCC/2"/>
+<wire x1="38.1" y1="167.64" x2="35.56" y2="167.64" width="0.1524" layer="91"/>
+<pinref part="⌁1" gate="G$1" pin="P$1"/>
+<wire x1="35.56" y1="167.64" x2="30.48" y2="167.64" width="0.1524" layer="91"/>
+<junction x="35.56" y="167.64"/>
+</segment>
 </net>
 <net name="PWR.MOTA" class="0">
@@
 <wire x1="274.32" y1="22.86" x2="264.16" y2="22.86" width="0.1524" layer="91"/>
 </segment>
-</net>
+<segment>
+<pinref part="X5" gate="G$1" pin="4"/>
+<pinref part="P+10" gate="1" pin="+5V"/>
+<wire x1="30.48" y1="160.02" x2="38.1" y2="160.02" width="0.1524" layer="91"/>
+<pinref part="⌁3" gate="G$1" pin="P$1"/>
+<wire x1="38.1" y1="160.02" x2="40.64" y2="160.02" width="0.1524" layer="91"/>
+<junction x="38.1" y="160.02"/>
+</segment>
+</net>

Commit message: wip baseboard quicksave  + now working on motor driver  + board area left is really, really tiny  + totally doable tough
Parts:
- removed X3: SYS-IIC, kitt.con:WüRTH-MINIB.VERTICAL
Connections:
- net N$2 renamed TOP.MOT-
- net N$4 renamed TOP.MOT+
Changed lines of the file:
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@@
 <part name="X1" library="kitt.con" deviceset="JST-4POS-2X" device="4POS"/>
 <part name="X2" library="kitt.con" deviceset="ROCKETBOARDS-LTC" device="TH" value="ATLAS-LTC"/>
-<part name="X3" library="kitt.con" deviceset="WüRTH-MINIB.VERTICAL" device="" value="SYS-IIC"/>
 <part name="X4" library="con-cypressindustries" deviceset="MINI-USB_SHIELD5P2-" device="32005-601" value="SYSTEWI"/>
 <part name="GND5" library="supply1" deviceset="GND" device=""/>
@@
 <instance part="X2" gate="X" x="120.65" y="58.42"/>
 <instance part="X2" gate="REF" x="118.11" y="58.42"/>
-<instance part="X3" gate="G$1" x="158.75" y="88.9" rot="R180"/>
 <instance part="X4" gate="G41" x="17.78" y="76.2" rot="MR0"/>
 <instance part="GND5" gate="1" x="25.4" y="63.5" rot="MR0"/>
@@
 </segment>
 </net>
-<net name="N$2" class="0">
+<net name="TOP.MOT-" class="0">
 <segment>
 <pinref part="SJ1" gate="G$1" pin="3"/>
@@
 </segment>
 </net>
-<net name="N$4" class="0">
+<net name="TOP.MOT+" class="0">
 <segment>
 <pinref part="X2.1" gate="-2" pin="1"/>
