File: Hardware/baseboard/eagle/main.sch (EAGLE design)
At the start: 34 parts, among them J1 MICROUSB-FEM, X1 JST-4POS-2X4POS, X1.2 TACH/LAP, X2 ATLAS-LTC, X2.1 MOTOR, X2.2 VRAILS+, X2.3 5V+SoC, X5 15244441

Commit message: wip baseboard  + schematic    -> finally added missing components    -> fixed some value spec mistakes  + layout    -> moved new components into areas where they fit best    -> probably moved some signals too, can't recall
Other:
- note removed: "[CAP MISSING?]"
Changed lines of the file:
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@@
 <part name="☇6" library="testpad" deviceset="PTR1" device="TP07SQ"/>
 <part name="☇9" library="testpad" deviceset="PTR1" device="TP07SQ"/>
-<part name="R1" library="kitt.psvs" deviceset="RKELV" device="1206" value="0.82R/⚻"/>
+<part name="R1" library="kitt.psvs" deviceset="RKELV" device="1206" value="8.2mR/⚻"/>
 <part name="U1" library="kitt.ic" deviceset="LTC4000" device="LTC4000EUFD#XXX"/>
 <part name="U$1" library="kitt.ic" deviceset="IRF7328" device=""/>
@@
 <part name="☇2" library="testpad" deviceset="PTR1" device="TP07SQ"/>
 <part name="R1" library="kitt.psvs" deviceset="RKELV" device="1206" value="15mR/25mW⚻"/>
+<part name="C4" library="rcl" deviceset="CPOL-EU" device="C/6032-28R" value="100uF"/>
+<part name="C5" library="rcl" deviceset="C-EU" device="C0402K" value="1uF/⇤"/>
 </parts>
 <sheets>
@@
 <text x="226.06" y="71.12" size="1.778" layer="115" ratio="20" align="center-left">[kerash]</text>
 <text x="210.82" y="116.84" size="1.778" layer="115" ratio="20" align="center-left">[domh]</text>
-<text x="40.64" y="149.86" size="1.778" layer="115" ratio="20" align="center-left">[CAP MISSING?]</text>
 </plain>
 <instances>
@@
 <instance part="☇2" gate="G$1" x="147.32" y="22.86" rot="MR270"/>
 <instance part="R1" gate="G$1" x="213.36" y="116.84" rot="MR0"/>
+<instance part="C4" gate="G$1" x="246.38" y="99.06"/>
+<instance part="C5" gate="G$1" x="53.34" y="73.66" smashed="yes" rot="MR0">
+<attribute name="NAME" x="50.546" y="72.771" size="1.778" layer="95" rot="MR0"/>
+<attribute name="VALUE" x="50.546" y="70.231" size="1.778" layer="96" rot="MR0"/>
+</instance>
 </instances>
 <busses>
@@
 <wire x1="228.6" y1="58.42" x2="228.6" y2="66.04" width="0.1524" layer="91"/>
 <junction x="177.8" y="58.42"/>
+<pinref part="C4" gate="G$1" pin="-"/>
+<wire x1="246.38" y1="93.98" x2="246.38" y2="58.42" width="0.1524" layer="91"/>
+<wire x1="246.38" y1="58.42" x2="228.6" y2="58.42" width="0.1524" layer="91"/>
+<junction x="228.6" y="58.42"/>
+<pinref part="C5" gate="G$1" pin="2"/>
+<wire x1="53.34" y1="68.58" x2="53.34" y2="58.42" width="0.1524" layer="91"/>
+<wire x1="53.34" y1="58.42" x2="68.58" y2="58.42" width="0.1524" layer="91"/>
+<junction x="68.58" y="58.42"/>
 </segment>
 <segment>
@@
 <segment>
 <pinref part="U1" gate="A" pin="ITH"/>
-<wire x1="73.66" y1="86.36" x2="48.26" y2="86.36" width="0.1524" layer="91"/>
-<label x="48.26" y="86.36" size="1.778" layer="95" rot="R180" xref="yes"/>
+<wire x1="73.66" y1="86.36" x2="30.48" y2="86.36" width="0.1524" layer="91"/>
+<label x="30.48" y="86.36" size="1.778" layer="95" rot="R180" xref="yes"/>
 </segment>
 <segment>
@@
 <pinref part="U1" gate="A" pin="VIN"/>
 <wire x1="91.44" y1="139.7" x2="91.44" y2="154.94" width="0.1524" layer="91"/>
-<wire x1="91.44" y1="154.94" x2="50.8" y2="154.94" width="0.1524" layer="91"/>
-<label x="50.8" y="154.94" size="1.778" layer="95" rot="R180" xref="yes"/>
+<wire x1="91.44" y1="154.94" x2="53.34" y2="154.94" width="0.1524" layer="91"/>
+<label x="22.86" y="154.94" size="1.778" layer="95" rot="R180" xref="yes"/>
 <pinref part="T1" gate="A" pin="D"/>
+<wire x1="53.34" y1="154.94" x2="22.86" y2="154.94" width="0.1524" layer="91"/>
 <wire x1="177.8" y1="132.08" x2="177.8" y2="154.94" width="0.1524" layer="91"/>
 <wire x1="177.8" y1="154.94" x2="91.44" y2="154.94" width="0.1524" layer="91"/>
@@
 <label x="96.52" y="157.48" size="1.778" layer="95" rot="R180"/>
 <label x="182.88" y="157.48" size="1.778" layer="95" rot="R180"/>
+<pinref part="C5" gate="G$1" pin="1"/>
+<wire x1="53.34" y1="76.2" x2="53.34" y2="154.94" width="0.1524" layer="91"/>
+<junction x="53.34" y="154.94"/>
 </segment>
 </net>
@@
 <pinref part="R2" gate="G$1" pin="1"/>
 <wire x1="218.44" y1="116.84" x2="228.6" y2="116.84" width="0.1524" layer="91"/>
-<wire x1="228.6" y1="116.84" x2="236.22" y2="116.84" width="0.1524" layer="91"/>
+<wire x1="228.6" y1="116.84" x2="246.38" y2="116.84" width="0.1524" layer="91"/>
 <junction x="228.6" y="116.84"/>
+<wire x1="246.38" y1="116.84" x2="251.46" y2="116.84" width="0.1524" layer="91"/>
 <wire x1="228.6" y1="116.84" x2="228.6" y2="99.06" width="0.1524" layer="91"/>
-<label x="236.22" y="116.84" size="1.778" layer="95" xref="yes"/>
+<label x="251.46" y="116.84" size="1.778" layer="95" xref="yes"/>
 <pinref part="R1" gate="G$1" pin="+"/>
+<pinref part="C4" gate="G$1" pin="+"/>
+<wire x1="246.38" y1="101.6" x2="246.38" y2="116.84" width="0.1524" layer="91"/>
+<junction x="246.38" y="116.84"/>
 </segment>
 </net>
@@
 <segment>
 <pinref part="U1" gate="A" pin="PLLIN/MODE"/>
-<wire x1="73.66" y1="96.52" x2="48.26" y2="96.52" width="0.1524" layer="91"/>
-<label x="48.26" y="96.52" size="1.778" layer="95" rot="R180" xref="yes"/>
+<wire x1="73.66" y1="96.52" x2="30.48" y2="96.52" width="0.1524" layer="91"/>
+<label x="30.48" y="96.52" size="1.778" layer="95" rot="R180" xref="yes"/>
 </segment>
 <segment>
@@
 <wire x1="73.66" y1="109.22" x2="66.04" y2="109.22" width="0.1524" layer="91"/>
 <wire x1="66.04" y1="109.22" x2="66.04" y2="106.68" width="0.1524" layer="91"/>
-<wire x1="66.04" y1="106.68" x2="48.26" y2="106.68" width="0.1524" layer="91"/>
-<label x="48.26" y="106.68" size="1.778" layer="95" rot="R180" xref="yes"/>
+<wire x1="66.04" y1="106.68" x2="30.48" y2="106.68" width="0.1524" layer="91"/>
+<label x="30.48" y="106.68" size="1.778" layer="95" rot="R180" xref="yes"/>
 </segment>
 <segment>
@@
 <segment>
 <pinref part="U1" gate="A" pin="RUN"/>
-<wire x1="73.66" y1="111.76" x2="48.26" y2="111.76" width="0.1524" layer="91"/>
-<label x="48.26" y="111.76" size="1.778" layer="95" rot="R180" xref="yes"/>
+<wire x1="73.66" y1="111.76" x2="30.48" y2="111.76" width="0.1524" layer="91"/>
+<label x="30.48" y="111.76" size="1.778" layer="95" rot="R180" xref="yes"/>
 </segment>
 <segment>
@@
 <segment>
 <pinref part="U1" gate="A" pin="PGOOD"/>
-<wire x1="73.66" y1="124.46" x2="50.8" y2="124.46" width="0.1524" layer="91"/>
-<label x="50.8" y="124.46" size="1.778" layer="95" rot="R180" xref="yes"/>
+<wire x1="73.66" y1="124.46" x2="30.48" y2="124.46" width="0.1524" layer="91"/>
+<label x="30.48" y="124.46" size="1.778" layer="95" rot="R180" xref="yes"/>
 </segment>
 <segment>
@@
 <part name="GND18" library="supply1" deviceset="GND" device=""/>
 <part name="L1" library="rcl" deviceset="L-EU" device="L2012C" value="BEAD"/>
-<part name="C1.1" library="rcl" deviceset="C-EU" device="C1210K" value="XX"/>
+<part name="C1" library="rcl" deviceset="C-EU" device="C1210K" value="10uF"/>
 <part name="F1" library="rcl" deviceset="R-EU_" device="R1210" value="1.5A-&gt;750mA "/>
 <part name="R3" library="rcl" deviceset="R-EU_" device="R0805W" value="10kR"/>
@@
 R1 = 10k
 A = R2/(R1+R2) -&gt; R2= ~ 2.2kR </text>
+<rectangle x1="78.74" y1="66.04" x2="91.44" y2="73.66" layer="116"/>
 </plain>
 <instances>
@@
 <instance part="GND18" gate="1" x="83.82" y="48.26"/>
 <instance part="L1" gate="G$1" x="72.39" y="83.82" rot="MR270"/>
-<instance part="C1.1" gate="G$1" x="83.82" y="71.12"/>
+<instance part="C1" gate="G$1" x="83.82" y="71.12"/>
 <instance part="F1" gate="G$1" x="116.84" y="83.82"/>
 <instance part="R3" gate="G$1" x="104.14" y="76.2" smashed="yes" rot="R90">
@@
 <pinref part="P+8" gate="1" pin="+18V"/>
 <pinref part="R3" gate="G$1" pin="2"/>
-<pinref part="C1.1" gate="G$1" pin="1"/>
+<pinref part="C1" gate="G$1" pin="1"/>
 <pinref part="L1" gate="G$1" pin="2"/>
 <pinref part="F1" gate="G$1" pin="1"/>
@@
 <junction x="104.14" y="53.34"/>
 <wire x1="104.14" y1="53.34" x2="132.08" y2="53.34" width="0.1524" layer="91"/>
-<pinref part="C1.1" gate="G$1" pin="2"/>
+<pinref part="C1" gate="G$1" pin="2"/>
 <pinref part="GND18" gate="1" pin="GND"/>
 <pinref part="R4" gate="G$1" pin="1"/>

Commit message: wip baseboard layout (keping airwires to 💯 edition)  + did some serious refactor in the LTC4000 area    -> flipped switch pinout again    -> gateswap on A5:U1    -> power polygons redrawn  + improvements include:    -> shorter SENSE distance (unexpected)    -> less vias as far as I recall
Connections:
- net +4.1V: now also S1.3; no longer S1.2
- net TOP.BAT/CON: now also S1.2; no longer S1.1
Other:
- moved on the sheet: S1
Changed lines of the file:
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@@
 <attribute name="NAME" x="86.36" y="132.08" size="1.4224" layer="95" ratio="5"/>
 </instance>
-<instance part="U$1" gate="A" x="132.08" y="144.78" rot="R90"/>
-<instance part="U$1" gate="B" x="205.74" y="116.84"/>
+<instance part="U$1" gate="A" x="205.74" y="116.84"/>
+<instance part="U$1" gate="B" x="132.08" y="144.78" rot="R90"/>
 </instances>
 <busses>
@@
 <junction x="134.62" y="134.62"/>
 <label x="137.16" y="137.16" size="1.778" layer="95" ratio="20" rot="R180"/>
-<pinref part="U$1" gate="A" pin="G"/>
+<pinref part="U$1" gate="B" pin="G"/>
 </segment>
 </net>
@@
 <wire x1="203.2" y1="86.36" x2="208.28" y2="86.36" width="0.1524" layer="91"/>
 <wire x1="208.28" y1="86.36" x2="220.98" y2="86.36" width="0.1524" layer="91"/>
-<wire x1="208.28" y1="86.36" x2="208.28" y2="111.76" width="0.1524" layer="91"/>
-<wire x1="208.28" y1="111.76" x2="165.1" y2="111.76" width="0.1524" layer="91"/>
+<wire x1="208.28" y1="86.36" x2="208.28" y2="109.22" width="0.1524" layer="91"/>
 <junction x="208.28" y="86.36"/>
 <pinref part="R8" gate="G$1" pin="2"/>
 <pinref part="U1" gate="X" pin="BAT"/>
-<pinref part="U$1" gate="B" pin="D"/>
-<junction x="208.28" y="111.76"/>
+<wire x1="205.74" y1="111.76" x2="165.1" y2="111.76" width="0.1524" layer="91"/>
+<wire x1="205.74" y1="111.76" x2="208.28" y2="109.22" width="0.1524" layer="91"/>
+<pinref part="U$1" gate="A" pin="D"/>
+<wire x1="208.28" y1="109.22" x2="208.28" y2="111.76" width="0.1524" layer="91"/>
+<junction x="208.28" y="109.22"/>
 </segment>
 </net>
@@
 <net name="CSN" class="0">
 <segment>
-<wire x1="165.1" y1="121.92" x2="208.28" y2="121.92" width="0.1524" layer="91"/>
-<wire x1="208.28" y1="132.08" x2="208.28" y2="121.92" width="0.1524" layer="91"/>
+<wire x1="165.1" y1="121.92" x2="205.74" y2="121.92" width="0.1524" layer="91"/>
+<wire x1="208.28" y1="132.08" x2="208.28" y2="124.46" width="0.1524" layer="91"/>
 <pinref part="R5" gate="G$1" pin="1"/>
 <pinref part="U1" gate="X" pin="CSN"/>
 <label x="175.26" y="124.46" size="1.778" layer="95" ratio="20" rot="R180"/>
-<pinref part="U$1" gate="B" pin="S"/>
-<junction x="208.28" y="121.92"/>
+<wire x1="205.74" y1="121.92" x2="208.28" y2="124.46" width="0.1524" layer="91"/>
+<pinref part="U$1" gate="A" pin="S"/>
+<wire x1="208.28" y1="121.92" x2="208.28" y2="124.46" width="0.1524" layer="91"/>
+<junction x="208.28" y="124.46"/>
 </segment>
 </net>
@@
 <wire x1="167.64" y1="119.38" x2="203.2" y2="119.38" width="0.1524" layer="91"/>
 <pinref part="U1" gate="X" pin="BGATE"/>
-<pinref part="U$1" gate="B" pin="G"/>
+<pinref part="U$1" gate="A" pin="G"/>
 </segment>
 </net>
@@
 <label x="121.92" y="154.94" size="1.778" layer="95" rot="R90" xref="yes"/>
 <pinref part="U1" gate="X" pin="IID"/>
-<pinref part="U$1" gate="A" pin="S"/>
-<wire x1="121.92" y1="147.32" x2="127" y2="147.32" width="0.1524" layer="91"/>
+<pinref part="U$1" gate="B" pin="S"/>
+<wire x1="127" y1="147.32" x2="121.92" y2="147.32" width="0.1524" layer="91"/>
 </segment>
 </net>
@@
 <net name="DDC.VOUT" class="0">
 <segment>
-<wire x1="139.7" y1="147.32" x2="149.86" y2="147.32" width="0.1524" layer="91"/>
+<wire x1="142.24" y1="147.32" x2="149.86" y2="147.32" width="0.1524" layer="91"/>
 <wire x1="149.86" y1="147.32" x2="149.86" y2="134.62" width="0.1524" layer="91"/>
-<wire x1="139.7" y1="144.78" x2="139.7" y2="147.32" width="0.1524" layer="91"/>
+<wire x1="139.7" y1="144.78" x2="142.24" y2="147.32" width="0.1524" layer="91"/>
 <wire x1="149.86" y1="147.32" x2="182.88" y2="147.32" width="0.1524" layer="91"/>
 <wire x1="182.88" y1="147.32" x2="182.88" y2="142.24" width="0.1524" layer="91"/>
@@
 <label x="154.94" y="149.86" size="1.778" layer="95" rot="R180"/>
 <pinref part="U1" gate="X" pin="CSP"/>
-<pinref part="U$1" gate="A" pin="D"/>
-<wire x1="137.16" y1="147.32" x2="139.7" y2="147.32" width="0.1524" layer="91"/>
-<junction x="139.7" y="147.32"/>
+<pinref part="U$1" gate="B" pin="D"/>
+<wire x1="137.16" y1="147.32" x2="142.24" y2="147.32" width="0.1524" layer="91"/>
+<junction x="142.24" y="147.32"/>
 </segment>
 </net>
@@
 </instance>
 <instance part="S3" gate="G$1" x="144.78" y="114.3" rot="MR0"/>
-<instance part="S1" gate="G$1" x="237.49" y="50.8"/>
+<instance part="S1" gate="G$1" x="238.76" y="50.8" rot="MR0"/>
 <instance part="P+4" gate="1" x="121.92" y="243.84" smashed="yes" rot="MR0">
 <attribute name="VALUE" x="120.65" y="245.11" size="1.778" layer="96" rot="MR90"/>
@@
 <wire x1="294.64" y1="66.04" x2="274.32" y2="66.04" width="0.1524" layer="91"/>
 <wire x1="274.32" y1="66.04" x2="274.32" y2="55.88" width="0.1524" layer="91"/>
-<wire x1="274.32" y1="55.88" x2="245.11" y2="55.88" width="0.1524" layer="91"/>
-<wire x1="245.11" y1="55.88" x2="245.11" y2="59.69" width="0.1524" layer="91"/>
-<wire x1="245.11" y1="59.69" x2="218.44" y2="59.69" width="0.1524" layer="91"/>
+<wire x1="274.32" y1="55.88" x2="250.19" y2="55.88" width="0.1524" layer="91"/>
+<wire x1="250.19" y1="55.88" x2="250.19" y2="59.69" width="0.1524" layer="91"/>
+<wire x1="250.19" y1="59.69" x2="218.44" y2="59.69" width="0.1524" layer="91"/>
 <pinref part="X1" gate="A" pin="2"/>
 <pinref part="X1" gate="B" pin="2"/>
@@
 <net name="TOP.BAT/CON" class="0">
 <segment>
-<pinref part="S1" gate="G$1" pin="1"/>
-<wire x1="247.65" y1="53.34" x2="274.32" y2="53.34" width="0.1524" layer="91"/>
-<wire x1="274.32" y1="53.34" x2="274.32" y2="45.72" width="0.1524" layer="91"/>
+<wire x1="248.92" y1="50.8" x2="274.32" y2="50.8" width="0.1524" layer="91"/>
+<wire x1="274.32" y1="50.8" x2="274.32" y2="45.72" width="0.1524" layer="91"/>
 <wire x1="274.32" y1="45.72" x2="294.64" y2="45.72" width="0.1524" layer="91"/>
 <wire x1="294.64" y1="45.72" x2="304.8" y2="45.72" width="0.1524" layer="91"/>
 <wire x1="304.8" y1="45.72" x2="304.8" y2="53.34" width="0.1524" layer="91"/>
-<label x="267.97" y="52.07" size="1.778" layer="95" ratio="20" rot="R180"/>
+<label x="267.97" y="54.61" size="1.778" layer="95" ratio="20" rot="R180"/>
 <pinref part="X1" gate="A" pin="1"/>
 <pinref part="D2" gate="G$1" pin="B"/>
 <wire x1="294.64" y1="48.26" x2="294.64" y2="45.72" width="0.1524" layer="91"/>
 <junction x="294.64" y="45.72"/>
+<pinref part="S1" gate="G$1" pin="2"/>
 </segment>
 </net>
@@
 <portref moduleinst="A5" port="BAT.+"/>
 <wire x1="215.9" y1="93.98" x2="215.9" y2="88.9" width="0.1524" layer="91"/>
-<pinref part="S1" gate="G$1" pin="2"/>
-<wire x1="215.9" y1="88.9" x2="215.9" y2="50.8" width="0.1524" layer="91"/>
-<wire x1="227.33" y1="50.8" x2="223.52" y2="50.8" width="0.1524" layer="91"/>
+<wire x1="215.9" y1="88.9" x2="215.9" y2="48.26" width="0.1524" layer="91"/>
 <pinref part="SUPPLY2" gate="P" pin="+4.1V"/>
-<wire x1="223.52" y1="50.8" x2="215.9" y2="50.8" width="0.1524" layer="91"/>
-<wire x1="223.52" y1="66.04" x2="223.52" y2="50.8" width="0.1524" layer="91"/>
-<junction x="223.52" y="50.8"/>
+<wire x1="228.6" y1="48.26" x2="223.52" y2="48.26" width="0.1524" layer="91"/>
+<wire x1="223.52" y1="48.26" x2="215.9" y2="48.26" width="0.1524" layer="91"/>
+<wire x1="223.52" y1="66.04" x2="223.52" y2="48.26" width="0.1524" layer="91"/>
+<junction x="223.52" y="48.26"/>
 <portref moduleinst="A10" port="VBAT"/>
 <wire x1="271.78" y1="93.98" x2="271.78" y2="88.9" width="0.1524" layer="91"/>
 <wire x1="271.78" y1="88.9" x2="215.9" y2="88.9" width="0.1524" layer="91"/>
 <junction x="215.9" y="88.9"/>
+<pinref part="S1" gate="G$1" pin="3"/>
 </segment>
 </net>
