File: Hardware/baseboard/eagle/main.sch (EAGLE design)
At the start: 34 parts, among them J1 MICROUSB-FEM, X1 JST-4POS-2X4POS, X1.2 TACH/LAP, X2 ATLAS-LTC, X2.1 MOTOR, X2.2 VRAILS+, X2.3 5V+SoC, X5 15244441

Commit message: wip baseboard: 50 airwires left  + schematic:    -> changed some resistor footprints, mostly pullup/pulldowns       and the megaohms voltage divider at the 1540  + layout:    -> new footprints of resistors had been moved to not overlap    -> expanded some powerlines in powerlayer, added vias etc
Parts:
- added L2: BEAD/0R/⎵, rcl:L-EUL2012C
- added R1: 100R, rcl:R-EU_R0402
Connections:
- new net A1: R1.2
- new net COM: R1.1
- new net COM.RRX: R1.1
- new net COMP: R1.1
- new net CTRL.A: R1.1
- new net DDC.CLN: R1.+
- new net DDC.OUT: R1.+
- new net DDC.VIN: R1.-
- new net EN0: R1.2
- new net INACT: R1.1
- new net N$4: D1.A2, R1.2
- new net REF: R1.2
- new net VDD: R1.1
- new net VOUT: R1.2
- new net ~SENSE+: R1.-
- new net ↔CLN: R1.K+
- new net ↔IN: R1.K-
- new net ↔SENSE+: R1.K+
- new net ↔SENSE-: R1.K-
- net !CS0: now also R1.2
- net +3V3: now also R1.1
- net +4.1V: now also R1.1; no longer D1.A2
- net +5V: now also D1.A1
- net GND: now also R1.2
- net N$1: now also R1.2
Other:
- note added: "removed because really close to output caps of 5VDCDC"
Changed lines of the file:
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@@
 <wire x1="203.2" y1="86.36" x2="208.28" y2="86.36" width="0.1524" layer="91"/>
 <wire x1="208.28" y1="86.36" x2="220.98" y2="86.36" width="0.1524" layer="91"/>
-<wire x1="208.28" y1="86.36" x2="208.28" y2="109.22" width="0.1524" layer="91"/>
+<wire x1="208.28" y1="86.36" x2="208.28" y2="111.76" width="0.1524" layer="91"/>
 <junction x="208.28" y="86.36"/>
 <pinref part="R8" gate="G$1" pin="2"/>
 <pinref part="U1" gate="X" pin="BAT"/>
-<wire x1="205.74" y1="111.76" x2="165.1" y2="111.76" width="0.1524" layer="91"/>
-<wire x1="205.74" y1="111.76" x2="208.28" y2="109.22" width="0.1524" layer="91"/>
+<wire x1="208.28" y1="111.76" x2="165.1" y2="111.76" width="0.1524" layer="91"/>
 <pinref part="U$1" gate="A" pin="D"/>
-<wire x1="208.28" y1="109.22" x2="208.28" y2="111.76" width="0.1524" layer="91"/>
-<junction x="208.28" y="109.22"/>
+<junction x="208.28" y="111.76"/>
 </segment>
 </net>
@@
 <net name="CSN" class="0">
 <segment>
-<wire x1="165.1" y1="121.92" x2="205.74" y2="121.92" width="0.1524" layer="91"/>
-<wire x1="208.28" y1="132.08" x2="208.28" y2="124.46" width="0.1524" layer="91"/>
+<wire x1="165.1" y1="121.92" x2="208.28" y2="121.92" width="0.1524" layer="91"/>
+<wire x1="208.28" y1="132.08" x2="208.28" y2="121.92" width="0.1524" layer="91"/>
 <pinref part="R5" gate="G$1" pin="1"/>
 <pinref part="U1" gate="X" pin="CSN"/>
 <label x="175.26" y="124.46" size="1.778" layer="95" ratio="20" rot="R180"/>
-<wire x1="205.74" y1="121.92" x2="208.28" y2="124.46" width="0.1524" layer="91"/>
 <pinref part="U$1" gate="A" pin="S"/>
-<wire x1="208.28" y1="121.92" x2="208.28" y2="124.46" width="0.1524" layer="91"/>
-<junction x="208.28" y="124.46"/>
+<junction x="208.28" y="121.92"/>
 </segment>
 </net>
@@
 <net name="DDC.VOUT" class="0">
 <segment>
-<wire x1="142.24" y1="147.32" x2="149.86" y2="147.32" width="0.1524" layer="91"/>
+<wire x1="139.7" y1="147.32" x2="149.86" y2="147.32" width="0.1524" layer="91"/>
 <wire x1="149.86" y1="147.32" x2="149.86" y2="134.62" width="0.1524" layer="91"/>
-<wire x1="139.7" y1="144.78" x2="142.24" y2="147.32" width="0.1524" layer="91"/>
+<wire x1="139.7" y1="144.78" x2="139.7" y2="147.32" width="0.1524" layer="91"/>
 <wire x1="149.86" y1="147.32" x2="182.88" y2="147.32" width="0.1524" layer="91"/>
 <wire x1="182.88" y1="147.32" x2="182.88" y2="142.24" width="0.1524" layer="91"/>
@@
 <pinref part="U1" gate="X" pin="CSP"/>
 <pinref part="U$1" gate="B" pin="D"/>
-<wire x1="137.16" y1="147.32" x2="142.24" y2="147.32" width="0.1524" layer="91"/>
-<junction x="142.24" y="147.32"/>
+<wire x1="137.16" y1="147.32" x2="139.7" y2="147.32" width="0.1524" layer="91"/>
+<junction x="139.7" y="147.32"/>
 </segment>
 </net>
@@
 <part name="GND1" library="supply1" deviceset="GND" device=""/>
 <part name="R3.1" library="rcl" deviceset="R-EU_" device="R0603" value="10kR/⎒"/>
-<part name="R3.2" library="rcl" deviceset="R-EU_" device="R0603" value="10kR/⎒"/>
-<part name="R3.3" library="rcl" deviceset="R-EU_" device="R0603" value="10kR/⎑"/>
-<part name="R3.4" library="rcl" deviceset="R-EU_" device="R0603" value="10kR/⎑"/>
-<part name="R3.5" library="rcl" deviceset="R-EU_" device="R0603" value="10kR/⎒"/>
-<part name="R3.6" library="rcl" deviceset="R-EU_" device="R0603" value="10kR/⎒"/>
+<part name="R3.2" library="rcl" deviceset="R-EU_" device="R0402" value="10kR/⎒"/>
+<part name="R3.3" library="rcl" deviceset="R-EU_" device="R0402" value="10kR/⎑"/>
+<part name="R3.4" library="rcl" deviceset="R-EU_" device="R0402" value="10kR/⎑"/>
+<part name="R3.5" library="rcl" deviceset="R-EU_" device="R0402" value="10kR/⎒"/>
+<part name="R3.6" library="rcl" deviceset="R-EU_" device="R0402" value="10kR/⎒"/>
 <part name="GND2" library="supply1" deviceset="GND" device=""/>
 <part name="GND3" library="supply1" deviceset="GND" device=""/>
@@
 <part name="R3.9" library="rcl" deviceset="R-EU_" device="R0603" value="60R/⇤"/>
 <part name="GND4" library="supply1" deviceset="GND" device=""/>
-<part name="R3.10" library="rcl" deviceset="R-EU_" device="R0603" value="10k/⎒"/>
-<part name="R3.11" library="rcl" deviceset="R-EU_" device="R0603" value="10kR/⎑"/>
+<part name="R3.10" library="rcl" deviceset="R-EU_" device="R0402" value="10k/⎒"/>
+<part name="R3.11" library="rcl" deviceset="R-EU_" device="R0402" value="10kR/⎑"/>
 <part name="+3V4" library="supply1" deviceset="+3V3" device=""/>
 <part name="GND5" library="supply1" deviceset="GND" device=""/>
@@
 <part name="R5" library="rcl" deviceset="R-EU_" device="R0402" value="10kR/⎒"/>
 <part name="R6" library="rcl" deviceset="R-EU_" device="R0402" value="10kR/⎒"/>
-<part name="C1" library="rcl" deviceset="C-EU" device="C0805K" value="100nF/⇤"/>
 </parts>
 <sheets>
@@
 <wire x1="137.16" y1="5.715" x2="142.24" y2="5.715" width="0.4064" layer="97"/>
 <text x="233.68" y="99.06" size="1.778" layer="97" ratio="20" align="center-left">{H}</text>
+<text x="86.36" y="40.64" size="1.778" layer="98">removed
+because
+really close to
+output caps of 5VDCDC</text>
 </plain>
 <instances>
@@
 <attribute name="VALUE" x="43.18" y="47.752" size="1.778" layer="96" rot="MR180"/>
 </instance>
-<instance part="C1" gate="G$1" x="93.98" y="45.72"/>
 </instances>
 <busses>
@@
 <label x="238.76" y="142.24" size="1.778" layer="95" ratio="20" xref="yes"/>
 <wire x1="99.06" y1="142.24" x2="238.76" y2="142.24" width="0.1524" layer="91"/>
-<pinref part="C1" gate="G$1" pin="1"/>
 <wire x1="93.98" y1="48.26" x2="93.98" y2="142.24" width="0.1524" layer="91"/>
 <junction x="93.98" y="142.24"/>
@@
 <wire x1="104.14" y1="33.02" x2="238.76" y2="33.02" width="0.1524" layer="91"/>
 <label x="238.76" y="33.02" size="1.778" layer="95" ratio="20" xref="yes"/>
-<pinref part="C1" gate="G$1" pin="2"/>
 <wire x1="93.98" y1="40.64" x2="93.98" y2="33.02" width="0.1524" layer="91"/>
 <junction x="93.98" y="33.02"/>
@@
 <part name="C1" library="rcl" deviceset="C-EU" device="C0402K" value="1uF/⇤"/>
 <part name="R2" library="rcl" deviceset="R-EU_" device="R0402" value="25kR"/>
-<part name="R3" library="rcl" deviceset="R-EU_" device="R0402" value="33MR"/>
-<part name="R4" library="rcl" deviceset="R-EU_" device="R0402" value="33MR"/>
+<part name="R3" library="rcl" deviceset="R-EU_" device="M0805" value="XXMR"/>
+<part name="R4" library="rcl" deviceset="R-EU_" device="M0805" value="XXMR"/>
 </parts>
 <sheets>
@@
 <part name="P+11" library="supply1" deviceset="+5V" device=""/>
 <part name="P+12" library="supply1" deviceset="+18V" device=""/>
+<part name="P+13" library="supply1" deviceset="+5V" device=""/>
+<part name="R1" library="rcl" deviceset="R-EU_" device="R0402" value="100R"/>
+<part name="L2" library="rcl" deviceset="L-EU" device="L2012C" value="BEAD/0R/⎵"/>
 </parts>
 <sheets>
@@
 <instance part="X2" gate="REF" x="119.38" y="58.42"/>
 <instance part="GND5" gate="1" x="25.4" y="63.5" rot="MR0"/>
-<instance part="SUPPLY3" gate="P" x="22.86" y="99.06"/>
+<instance part="SUPPLY3" gate="P" x="12.7" y="101.6"/>
 <instance part="D1" gate="G$1" x="33.02" y="91.44" rot="R180"/>
 <instance part="GND7" gate="1" x="93.98" y="43.18" rot="MR0"/>
@@
 <attribute name="VALUE" x="101.6" y="142.24" size="1.778" layer="96" rot="R180"/>
 </instance>
+<instance part="P+13" gate="1" x="40.64" y="101.6" smashed="yes" rot="MR0">
+<attribute name="VALUE" x="40.005" y="102.235" size="1.778" layer="96" rot="MR90"/>
+</instance>
+<instance part="R1" gate="G$1" x="20.32" y="91.44"/>
+<instance part="L2" gate="G$1" x="152.4" y="149.86" smashed="yes" rot="R270">
+<attribute name="NAME" x="148.59" y="151.3586" size="1.778" layer="95"/>
+<attribute name="VALUE" x="148.59" y="146.558" size="1.778" layer="96"/>
+</instance>
 </instances>
 <busses>
@@
 <wire x1="91.44" y1="134.62" x2="99.06" y2="129.54" width="0.1524" layer="91"/>
 </segment>
+<segment>
+<pinref part="P+13" gate="1" pin="+5V"/>
+<pinref part="D1" gate="G$1" pin="A1"/>
+<wire x1="40.64" y1="99.06" x2="40.64" y2="91.44" width="0.1524" layer="91"/>
+<wire x1="40.64" y1="91.44" x2="38.1" y2="91.44" width="0.1524" layer="91"/>
+</segment>
 </net>
 <net name="UNO.5V" class="0">
@@
 <segment>
 <pinref part="SUPPLY3" gate="P" pin="+4.1V"/>
-<pinref part="D1" gate="G$1" pin="A2"/>
-<wire x1="22.86" y1="96.52" x2="22.86" y2="91.44" width="0.1524" layer="91"/>
-<wire x1="22.86" y1="91.44" x2="27.94" y2="91.44" width="0.1524" layer="91"/>
+<wire x1="12.7" y1="99.06" x2="12.7" y2="91.44" width="0.1524" layer="91"/>
+<pinref part="R1" gate="G$1" pin="1"/>
+<wire x1="15.24" y1="91.44" x2="12.7" y2="91.44" width="0.1524" layer="91"/>
 </segment>
 <segment>
@@
 </segment>
 </net>
+<net name="N$4" class="0">
+<segment>
+<pinref part="R1" gate="G$1" pin="2"/>
+<pinref part="D1" gate="G$1" pin="A2"/>
+<wire x1="25.4" y1="91.44" x2="27.94" y2="91.44" width="0.1524" layer="91"/>
+</segment>
+</net>

Commit message: baseboard  + layout    -> some progress (+6 airwires done)  + schematic    -> added todo item in LTC1540 subassembly regarding bias
Other:
- note added: "High side PMOS gate:"
- note added: "VIN and IOREF are Outpus"
- note added: "[TODO] Add Logic/transistors for a; a bias in case the battery is not connected b; when the comparator shuts off when the battery is connected c; when the system managment might want to override"
- note added: "tie to 3v3 from ghostcar bb20"
Changed lines of the file:
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@@
 Package?
 Seems unlikely a 33MR will be a 0402</text>
+<text x="182.88" y="83.82" size="1.778" layer="98">[TODO]
+Add Logic/transistors for
+a; a bias in case the battery is not connected
+b; when the comparator shuts off when the battery is connected
+c; when the system managment might want to override</text>
+<wire x1="218.44" y1="96.52" x2="228.6" y2="101.6" width="0.1524" layer="98"/>
+<wire x1="228.6" y1="101.6" x2="231.14" y2="109.22" width="0.1524" layer="98"/>
+<wire x1="231.14" y1="109.22" x2="231.14" y2="114.3" width="0.1524" layer="98"/>
+<wire x1="231.14" y1="114.3" x2="226.06" y2="119.38" width="0.1524" layer="98"/>
+<wire x1="226.06" y1="119.38" x2="208.28" y2="124.46" width="0.1524" layer="98"/>
+<wire x1="208.28" y1="124.46" x2="200.66" y2="124.46" width="0.1524" layer="98"/>
+<wire x1="200.66" y1="124.46" x2="193.04" y2="127" width="0.1524" layer="98"/>
+<wire x1="193.04" y1="127" x2="193.04" y2="124.46" width="0.1524" layer="98"/>
+<wire x1="193.04" y1="124.46" x2="198.12" y2="127" width="0.1524" layer="98"/>
+<wire x1="198.12" y1="127" x2="193.04" y2="127" width="0.1524" layer="98"/>
+<text x="213.36" y="96.52" size="1.778" layer="98">High side PMOS gate:</text>
 </plain>
 <instances>
@@
 <text x="99.06" y="30.48" size="1.9304" layer="98">Question:
 [an##]: annotation##  or anton##?</text>
+<text x="7.62" y="142.24" size="1.778" layer="98" rot="R90">VIN and IOREF are Outpus</text>
+<text x="30.48" y="165.1" size="1.778" layer="98">tie to 3v3 from ghostcar bb20</text>
 </plain>
 <instances>

Commit message: wip baseboard  -> layout: did some easy airwires
Other:
- note added: "Pin2 really N/C?"
Changed lines of the file:
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@@
 <wire x1="198.12" y1="127" x2="193.04" y2="127" width="0.1524" layer="98"/>
 <text x="213.36" y="96.52" size="1.778" layer="98">High side PMOS gate:</text>
+<text x="165.1" y="116.84" size="1.778" layer="98">Pin2 really N/C?
+</text>
 </plain>
 <instances>

Commit message: wip baseboard layout quicksave  + schematic    -> revised high side guard, added NAND logic  + layout    -> moved entire guard circuit on north west corner,       ideal fit acutally. Spooky how this works.    -> redo of input protection and powerlines,       make slightly more sense now
Parts:
- removed ⌁1: SINGLEPAD40MIL-BREAK.PILOT, kitt.con:SINGLEPAD40MIL-BREAK.PILOT
- removed ⌁2, ⌁3: SINGLEPAD40MIL-BREAK, kitt.con:SINGLEPAD40MIL-BREAK
- added ☇1: 1, kitt.con:CON.BUOC.IOBPD-P5MM
- added ☇10: 10, kitt.con:CON.BUOC.IOBPD-P5MM
- added ☇2: 2, kitt.con:CON.BUOC.IOBPD-P5MM
- added ☇3: 3, kitt.con:CON.BUOC.IOBPD-P5MM
- added ☇4: 4, kitt.con:CON.BUOC.IOBPD-P5MM
- added ☇5: 5, kitt.con:CON.BUOC.IOBPD-P5MM
- added ☇6: 6, kitt.con:CON.BUOC.IOBPD-P5MM
- added ☇7: 7, kitt.con:CON.BUOC.IOBPD-P5MM
- added ☇8: 8, kitt.con:CON.BUOC.IOBPD-P5MM
- added ☇9: 9, kitt.con:CON.BUOC.IOBPD-P5MM
- added ☇XX1.1: VRAILS, kitt.con:CON.BUOC.IOBPD-P5MM
- added ☇XX1.2, ☇XX1.3: GND, kitt.con:CON.BUOC.IOBPD-P5MM
- added ☇XX1.4: +5V, kitt.con:CON.BUOC.IOBPD-P5MM
Connections:
- removed net V++: ⌁2.P$1
- new net CL: ☇6.TP
- new net CTRL.ENC: ☇2.TP
- new net CTRL.FREQ: ☇6.TP
- new net CTRL.PGOOD: ☇7.TP
- new net CTRL.PLLIN/MODE: ☇9.TP
- new net CTRL.RUN: ☇8.TP
- new net DDC.EXTVCC: ☇1.TP
- new net DDC.ITH: ☇2.TP
- new net DRDY_M: ☇1.TP
- new net IBMON: ☇7.TP
- new net IIMON: ☇8.TP
- new net IL: ☇3.TP
- new net INT2_AG: ☇3.TP
- new net INT_M: ☇2.TP
- new net TMR: ☇1.TP
- new net ↔FBG: ☇4.TP
- net !CS1: now also X2X.14, ☇10.P$1
- net +3V3: now also X2X.10, X2X.2
- net +5V: now also ☇XX1.4.P$1; no longer ⌁3.P$1
- net +9V: now also X2X.1
- net DDC.CLN: now also ☇9.TP
- net DDC.OUT: now also ☇3.TP
- net DDC.VIN: now also ☇5.TP
- net GND: now also X2.2-2.1, ☇XX1.2.P$1, ☇XX1.3.P$1; no longer X2.2-1.1, ⌁1.P$1, ⌁2.P$1
- net MISO: now also X2X.5
- net MOSI: now also X2X.6
- net VCC/2: now also X2.2-1.1, ☇XX1.1.P$1; no longer X2.2-2.1, ⌁1.P$1
- net VSYS: no longer ⌁3.P$1
- net ~SENSE+: now also ☇4.TP
- net ↔ILIM: now also ☇5.TP
Other:
- note added: "2.4 - 3.5 V (LOW POWER!)"
- note added: "4.2-4.35V"
- note added: "??? ???"
- note added: "Battery Guard Circuit / Contactor"
- note added: "Build your Own Connector"
- note added: "CMOS LOGIC LEVEL"
- note added: "ESD'16 PROJECT G2 / "Carrera AI""
- note added: "IID"
- note added: "KITT-MK1"
- note added: "Kit for Intelligent, Trainable Trackcars"
- note added: "SCHEMATICS"
- note added: "Schmitt-Triggered HIGH: 2.0V to VDD"
- note added: "[ANNOTATION] The Quick Brown Fox Jumps Over The Lazy Dog"
- note removed: "Battery Voltage Guard Circuit"
- note removed: "High side PMOS gate:"
- note removed: "Pin2 really N/C?"
- note removed: "Question: [an##]: annotation## or anton##?"
- note removed: "TODO: Put into submodule before route -> crowded either that or use A3"
- note removed: "[TODO] Add Logic/transistors for a; a bias in case the battery is not connected b; when the comparator shuts off when the battery is connected c; when the system managment might want to override"
- note removed: "[spc1]"
- note removed: "[spc1] Inductor Part Specs: Taiyo Yuden NRS8030T4R7MJGJ ESR: 28.6 mOhm max I_sat = 3.6A I_max = 4A f_res = 40MHz Digikey# 587-2969-1-ND"
- note removed: "[todo] Package? Seems unlikely a 33MR will be a 0402"

Commit message: wip baseboard layout  + just now realized/looked up that I've had plans    initially to extend the north/south edge of the board area    which makes the jumper situation really easy  + motor is now connected via a jumper wire  + reminder that this design is still smaller    than a credit card  + pretty much finished on battery guard
Parts:
- added F2: (no value), fuse:SH22
- added JP1, JP2: (no value), pinhead:PINHD-1X1
- added PAD1, PAD2: WIREPADSMD2,54-5,08, wirepad:WIREPADSMD2,54-5,08
Connections:
- new net TOP.18V/PREFUSE: F2.1, JP1.1, PAD1.P
- net +18V: now also F2.2, JP2.1, PAD2.P
- net +5V: now also D1.A2; no longer D1.A1
- net N$4: now also D1.A1; no longer D1.A2
Other:
- moved on the sheet: SJ1, X2.1-1, X2.1-2, X2.2-2
