File: Hardware/baseboard/eagle/baseboard.sch (EAGLE design)
At the start: 41 parts, among them J1 MICROUSB-FEM, X1 JST-4POS-2X4POS, X1.2 TACH/LAP, X2.2 VRAILS+, X2.3 5V+SoC

Commit message: Final Layout
Other:
- moved on the sheet: TP2, TP3
Changed lines of the file:
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@@
 <instance part="X2" gate="-2" x="53.34" y="20.32" rot="R180"/>
 <instance part="X2" gate="-3" x="53.34" y="53.34" rot="R180"/>
-<instance part="TP2" gate="G$1" x="304.8" y="210.82" rot="R180"/>
-<instance part="TP3" gate="G$1" x="309.88" y="210.82" rot="R180"/>
+<instance part="TP2" gate="G$1" x="304.8" y="203.2" rot="R180"/>
+<instance part="TP3" gate="G$1" x="309.88" y="203.2" rot="R180"/>
 <instance part="TP4" gate="G$1" x="314.96" y="210.82" rot="R180"/>
 <instance part="TP5" gate="G$1" x="320.04" y="210.82" rot="R180"/>
@@
 <segment>
 <pinref part="TP2" gate="G$1" pin="TP"/>
-<wire x1="304.8" y1="213.36" x2="304.8" y2="218.44" width="0.1524" layer="91"/>
+<wire x1="304.8" y1="205.74" x2="304.8" y2="218.44" width="0.1524" layer="91"/>
 </segment>
 </net>
@@
 <segment>
 <pinref part="TP3" gate="G$1" pin="TP"/>
-<wire x1="309.88" y1="213.36" x2="309.88" y2="218.44" width="0.1524" layer="91"/>
-</segment>
-</net>
+<wire x1="309.88" y1="205.74" x2="309.88" y2="218.44" width="0.1524" layer="91"/>
+</segment>
+</net>

Commit message: updated schematic
Parts:
- removed GUIDE1: BREAK.GUIDE40MIL-BREAK, kitt.con:BREAK.GUIDE40MIL-BREAK
- removed REF1: EAGLE EDU LIMIT, kitt.refs:REF.EDULIMIT
- removed REF2: REF.LOGO.UASUA, kitt.refs:REF.LOGO.UASUA
Connections:
- net TOP.V+PWR renamed +24V
Other:
- note removed: "[q1] Buffer cap? why not here?"
- note removed: "⇽ CURRENT ⇽"
- moved on the sheet: D2, L1, L2, L5, X1A, X1B
