File: Hardware/baseboard/eagle/CarrerAI_BB_V1.0.sch (EAGLE design)
At the start: 38 parts, among them J1 MICROUSB-FEM, X1 JST-4POS-2X4POS, X1.2 TACH/LAP, X2.2 VRAILS+, X2.3 5V+SoC

Commit message: BB-SRII: pretty much, out of the blue, the gyro area opti/minimized itself
looks nice
Parts:
- removed TP2, TP3, TP4, TP5, TP6, TP7: TPTP07R, testpad:TPTP07R
- added X5: 87758-0816, con-molex:87758-0816
- added X6: 87758-0616, con-molex:87758-0616
Connections:
- removed net TOP1: TP2.TP
- removed net TOP2: TP3.TP
- removed net TOP3: TP4.TP
- removed net TOP4: TP5.TP
- removed net TOP5: TP6.TP
- removed net TOP6: TP7.TP
- net +3V3: now also X6-5.S, X6-6.S
- net N$3: no longer TP2.TP
- net N$4: no longer TP3.TP
- net N$5: no longer TP4.TP
Other:
- note added: "Prototype Interception"
- note added: "[note]: can patch together IRQs into VIA"
- note added: "«gumstick»"
- note removed: "Power Control & Monitor Unit"

Commit message: BB-SRII: minor fixes, in process of dropping the fat good for nothin' pmos
the weather is nice outside
Connections:
- new net A10.!ACT: X5-7.S
- new net TOP.5VEN: X5-3.S
- new net TOP.PGOOD: X6-1.S
- new net TOP.RUN: X6-2.S
- new net TOP.VSYS/GUARD: X5-1.S
- net +5V: now also X5-2.S
- net GND: now also X5-4.S, X5-6.S, X5-8.S
- net TOP.!RST: now also X6-4.S
Other:
- note added: "TODO: add manual override patchthrough at top level TODO: add classic 1M:10k PUPD resistors"
- moved on the sheet: X5-1, X6-1, X6-2, X6-3, X6-4
Changed lines of the file:
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@@
 Optional Current Programming Resistor
 Populate with Capacitor and fitting value</text>
+<text x="43.18" y="48.26" size="1.778" layer="90">TODO: add manual override patchthrough at top level
+TODO: add classic 1M:10k PUPD resistors </text>
 </plain>
 <instances>
@@
 <part name="FRAME1" library="frames" deviceset="A4L-LOC" device=""/>
 <part name="U1" library="kitt.ic" deviceset="LTC1540" device="CDD-LONG"/>
-<part name="T1" library="kitt.ic" deviceset="SI4427BDY" device=""/>
 <part name="GND1" library="supply1" deviceset="GND" device=""/>
 <part name="R7" library="rcl" deviceset="R-EU_" device="R0402" value="2.32MR"/>
@@
 <instance part="FRAME1" gate="G$1" x="0" y="0"/>
 <instance part="U1" gate="U" x="114.3" y="104.14"/>
-<instance part="T1" gate="G$1" x="175.26" y="134.62" smashed="yes" rot="R90">
-<attribute name="VALUE" x="171.45" y="140.97" size="1.778" layer="96"/>
-<attribute name="NAME" x="171.45" y="143.51" size="1.778" layer="95"/>
-</instance>
 <instance part="GND1" gate="1" x="114.3" y="40.64"/>
 <instance part="R7" gate="G$1" x="53.34" y="71.12" rot="R90"/>
@@
 </busses>
 <nets>
-<net name="POW.SINK" class="0">
-<segment>
-<pinref part="T1" gate="G$1" pin="D"/>
-<wire x1="180.34" y1="137.16" x2="220.98" y2="137.16" width="0.1524" layer="91"/>
-<label x="220.98" y="137.16" size="1.778" layer="95" xref="yes"/>
-</segment>
-</net>
 <net name="VBAT" class="0">
 <segment>
@@
 <net name="POW.SRC" class="0">
 <segment>
-<pinref part="T1" gate="G$1" pin="S"/>
-<wire x1="170.18" y1="137.16" x2="144.78" y2="137.16" width="0.1524" layer="91"/>
 <label x="33.02" y="137.16" size="1.778" layer="95" rot="R180" xref="yes"/>
 <pinref part="U1" gate="U" pin="V+"/>
@@
 <wire x1="144.78" y1="81.28" x2="144.78" y2="137.16" width="0.1524" layer="91"/>
 <junction x="144.78" y="137.16"/>
+<wire x1="144.78" y1="137.16" x2="220.98" y2="137.16" width="0.1524" layer="91"/>
+<label x="220.98" y="137.16" size="1.778" layer="95" xref="yes"/>
 </segment>
 </net>
@@
 <segment>
 <label x="220.98" y="124.46" size="1.778" layer="95" xref="yes"/>
-<pinref part="T1" gate="G$1" pin="G"/>
 <wire x1="220.98" y1="124.46" x2="205.74" y2="124.46" width="0.1524" layer="91"/>
-<wire x1="172.72" y1="124.46" x2="172.72" y2="132.08" width="0.1524" layer="91"/>
 <wire x1="205.74" y1="99.06" x2="205.74" y2="124.46" width="0.1524" layer="91"/>
-<wire x1="205.74" y1="124.46" x2="172.72" y2="124.46" width="0.1524" layer="91"/>
-<junction x="205.74" y="124.46"/>
 <pinref part="U2" gate="1" pin="Y"/>
 <wire x1="205.74" y1="99.06" x2="187.96" y2="99.06" width="0.1524" layer="91"/>
@@
 <part name="X6" library="con-molex" deviceset="87758-0616" device=""/>
 <part name="+3V8" library="supply1" deviceset="+3V3" device=""/>
+<part name="GND7" library="supply1" deviceset="GND" device=""/>
+<part name="VDD1" library="supply1" deviceset="VDD" device="" value="NOT VSYS ANYMORE"/>
 </parts>
 <sheets>
@@
 <instance part="SUPPLY2" gate="P" x="200.66" y="66.04"/>
 <instance part="D2" gate="G$1" x="254" y="53.34"/>
-<instance part="P+11" gate="1" x="330.2" y="200.66" smashed="yes">
-<attribute name="VALUE" x="332.74" y="203.2" size="1.778" layer="96" rot="R180"/>
+<instance part="P+11" gate="1" x="431.8" y="200.66" smashed="yes">
+<attribute name="VALUE" x="434.34" y="203.2" size="1.778" layer="96" rot="R180"/>
 </instance>
 <instance part="JP1" gate="G$1" x="91.44" y="86.36" rot="R270"/>
@@
 <attribute name="VALUE" x="96.52" y="241.3" size="1.778" layer="96" rot="R90"/>
 </instance>
-<instance part="X5" gate="-1" x="419.1" y="180.34"/>
+<instance part="X5" gate="-1" x="419.1" y="180.34" rot="MR0"/>
 <instance part="X5" gate="-2" x="439.42" y="180.34"/>
 <instance part="X5" gate="-3" x="419.1" y="177.8"/>
@@
 <instance part="X5" gate="-7" x="419.1" y="172.72"/>
 <instance part="X5" gate="-8" x="439.42" y="172.72"/>
-<instance part="X6" gate="-1" x="421.64" y="226.06" rot="MR0"/>
-<instance part="X6" gate="-2" x="441.96" y="226.06"/>
-<instance part="X6" gate="-3" x="421.64" y="223.52" rot="MR0"/>
-<instance part="X6" gate="-4" x="441.96" y="223.52"/>
+<instance part="X6" gate="-1" x="421.64" y="226.06"/>
+<instance part="X6" gate="-2" x="441.96" y="226.06" rot="MR0"/>
+<instance part="X6" gate="-3" x="421.64" y="223.52"/>
+<instance part="X6" gate="-4" x="441.96" y="223.52" rot="MR0"/>
 <instance part="X6" gate="-5" x="421.64" y="220.98" rot="MR0"/>
 <instance part="X6" gate="-6" x="441.96" y="220.98"/>
@@
 <attribute name="VALUE" x="432.435" y="234.315" size="1.778" layer="96" rot="R90"/>
 </instance>
+<instance part="GND7" gate="1" x="431.8" y="165.1"/>
+<instance part="VDD1" gate="G$1" x="292.1" y="96.52" smashed="yes" rot="R180"/>
 </instances>
 <busses>
@@
 <pinref part="GND3" gate="1" pin="GND"/>
 </segment>
+<segment>
+<pinref part="GND7" gate="1" pin="GND"/>
+<pinref part="X5" gate="-4" pin="S"/>
+<wire x1="431.8" y1="167.64" x2="431.8" y2="172.72" width="0.1524" layer="91"/>
+<wire x1="431.8" y1="172.72" x2="431.8" y2="175.26" width="0.1524" layer="91"/>
+<wire x1="431.8" y1="175.26" x2="431.8" y2="177.8" width="0.1524" layer="91"/>
+<wire x1="431.8" y1="177.8" x2="436.88" y2="177.8" width="0.1524" layer="91"/>
+<pinref part="X5" gate="-6" pin="S"/>
+<wire x1="436.88" y1="175.26" x2="431.8" y2="175.26" width="0.1524" layer="91"/>
+<junction x="431.8" y="175.26"/>
+<pinref part="X5" gate="-8" pin="S"/>
+<wire x1="436.88" y1="172.72" x2="431.8" y2="172.72" width="0.1524" layer="91"/>
+<junction x="431.8" y="172.72"/>
+</segment>
 </net>
 <net name="+18V" class="0">
@@
 <segment>
 <pinref part="P+11" gate="1" pin="+5V"/>
-<wire x1="330.2" y1="198.12" x2="330.2" y2="193.04" width="0.1524" layer="91"/>
+<pinref part="X5" gate="-2" pin="S"/>
+<wire x1="431.8" y1="198.12" x2="431.8" y2="180.34" width="0.1524" layer="91"/>
+<wire x1="431.8" y1="180.34" x2="436.88" y2="180.34" width="0.1524" layer="91"/>
 </segment>
 </net>
@@
 <label x="236.22" y="185.42" size="1.778" layer="95" ratio="20" rot="R180"/>
 </segment>
+<segment>
+<wire x1="444.5" y1="226.06" x2="462.28" y2="226.06" width="0.1524" layer="91"/>
+<label x="459.74" y="228.6" size="1.778" layer="95" rot="R180"/>
+<pinref part="X6" gate="-2" pin="S"/>
+</segment>
 </net>
 <net name="TOP.FREQ" class="0">
@@
 <label x="236.22" y="175.26" size="1.778" layer="95" ratio="20" rot="R180"/>
 </segment>
+<segment>
+<wire x1="467.36" y1="203.2" x2="449.58" y2="203.2" width="0.1524" layer="91"/>
+</segment>
 </net>
 <net name="TOP.PGOOD" class="0">
@@
 <wire x1="297.18" y1="177.8" x2="218.44" y2="177.8" width="0.1524" layer="91"/>
 <label x="236.22" y="180.34" size="1.778" layer="95" ratio="20" rot="R180"/>
+</segment>
+<segment>
+<wire x1="419.1" y1="226.06" x2="401.32" y2="226.06" width="0.1524" layer="91"/>
+<label x="416.56" y="228.6" size="1.778" layer="95" rot="R180"/>
+<pinref part="X6" gate="-1" pin="S"/>
 </segment>
 </net>
@@
 <portref moduleinst="A7" port="!RESET"/>
 </segment>
+<segment>
+<wire x1="444.5" y1="223.52" x2="462.28" y2="223.52" width="0.1524" layer="91"/>
+<pinref part="X6" gate="-4" pin="S"/>
+<label x="452.12" y="220.98" size="1.778" layer="95"/>
+</segment>
 </net>
 <net name="VDD" class="0">
@@
 <wire x1="100.33" y1="228.6" x2="91.44" y2="228.6" width="0.1524" layer="91"/>
 <portref moduleinst="A7" port="VSYS"/>
+</segment>
+<segment>
+<portref moduleinst="A9" port="VIN"/>
+<portref moduleinst="A10" port="POW.SINK"/>
+<wire x1="287.02" y1="104.14" x2="292.1" y2="104.14" width="0.1524" layer="91"/>
+<pinref part="VDD1" gate="G$1" pin="VDD"/>
+<wire x1="292.1" y1="104.14" x2="297.18" y2="104.14" width="0.1524" layer="91"/>
+<wire x1="292.1" y1="99.06" x2="292.1" y2="104.14" width="0.1524" layer="91"/>
+<junction x="292.1" y="104.14"/>
 </segment>
 </net>
@@
 <net name="TOP.VSYS/GUARD" class="0">
 <segment>
-<portref moduleinst="A9" port="VIN"/>
-<portref moduleinst="A10" port="POW.SINK"/>
-<wire x1="287.02" y1="104.14" x2="292.1" y2="104.14" width="0.1524" layer="91"/>
-<portref moduleinst="A9" port="EN"/>
-<wire x1="292.1" y1="104.14" x2="297.18" y2="104.14" width="0.1524" layer="91"/>
-<wire x1="297.18" y1="111.76" x2="292.1" y2="111.76" width="0.1524" layer="91"/>
-<wire x1="292.1" y1="111.76" x2="292.1" y2="104.14" width="0.1524" layer="91"/>
-<junction x="292.1" y="104.14"/>
-</segment>
-<segment>
 <wire x1="289.56" y1="73.66" x2="299.72" y2="73.66" width="0.1524" layer="91"/>
+</segment>
+<segment>
+<wire x1="426.72" y1="193.04" x2="426.72" y2="180.34" width="0.1524" layer="91"/>
+<wire x1="426.72" y1="193.04" x2="419.1" y2="193.04" width="0.1524" layer="91"/>
+<label x="419.1" y="193.04" size="1.778" layer="95" rot="R180" xref="yes"/>
+<wire x1="426.72" y1="180.34" x2="421.64" y2="180.34" width="0.1524" layer="91"/>
+<pinref part="X5" gate="-1" pin="S"/>
 </segment>
 </net>
@@
 <label x="292.1" y="129.54" size="1.778" layer="95" rot="R90"/>
 </segment>
+<segment>
+<label x="411.48" y="175.26" size="1.778" layer="95" rot="R180"/>
+<wire x1="416.56" y1="172.72" x2="401.32" y2="172.72" width="0.1524" layer="91"/>
+<pinref part="X5" gate="-7" pin="S"/>
+</segment>
 </net>
 <net name="TOP.!BATOK" class="0">
@@
 </segment>
 </net>
+<net name="TOP.5VEN" class="0">
+<segment>
+<portref moduleinst="A9" port="EN"/>
+<wire x1="297.18" y1="111.76" x2="297.18" y2="119.38" width="0.1524" layer="91"/>
+<wire x1="297.18" y1="119.38" x2="299.72" y2="119.38" width="0.1524" layer="91"/>
+<wire x1="299.72" y1="119.38" x2="299.72" y2="139.7" width="0.1524" layer="91"/>
+<wire x1="299.72" y1="139.7" x2="314.96" y2="139.7" width="0.1524" layer="91"/>
+<wire x1="314.96" y1="139.7" x2="314.96" y2="152.4" width="0.1524" layer="91"/>
+<label x="312.42" y="142.24" size="1.778" layer="95" rot="R180"/>
+</segment>
+<segment>
+<wire x1="401.32" y1="177.8" x2="416.56" y2="177.8" width="0.1524" layer="91"/>
+<pinref part="X5" gate="-3" pin="S"/>
+</segment>
+</net>

Commit message: CarrerAI BB SV2: it dowsn't look like much has changed but there has been some progress.
Parts:
- removed J1: MICROUSB-FEM, kitt.con:MICROUSB-FEM
- added LED1: VINS, led:LEDCHIP-LED0805
- added LED2: VSYS, led:LEDCHIP-LED0805
- added LED3: 5VCC, led:LEDCHIP-LED0805
- added LED4: 3VCC, led:LEDCHIP-LED0805
- added LED5: PROBLEM, led:LEDCHIP-LED0805
- added PAD1, PAD2: (no value), wirepad:1,6/0,9
- added R8: 100R, rcl:R-EU_R0402
- added SV3: (no value), con-lsta:FE05-2W
- added X3: 87758-1016, con-molex:87758-1016
- X2.3: value 5V+SoC -> SoC
Connections:
- net N$7 renamed UNO.ADC3
- net N$9 renamed UNO.ADC1
- net VBAT renamed VSYS
- removed net +24V: JP1.1, L4.1
- removed net A0: R5.2, R6.1
- removed net A1: R1.2, R2.1
- removed net A2: R3.2, R4.1
- removed net REF: R1.2, R2.1
- removed net TOP.VSYS/GUARD: X5-1.S
- new net BAT.+: R8.2
- new net IN+&REF: R1.2, R2.1
- new net TOP.FREQ: X5-5.S
- new net TOP.MODE: X6-3.S
- new net UNO.ADC2: XA1G$1.ADC.2, ☈2.2
- net !CS1: now also R8.2
- net !PD: now also R8.1
- net +18V: now also JP1.1, L4.1, PAD1.P, PAD2.P
- net +3V3: now also X1-2.S; no longer J1.1
- net EN: now also R4.1, R5.1, R5.2
- net GND: no longer J1.GND, J1.S, R4.2, R6.2
- net N$1: no longer J1.VBUS
- net N$8: now also R8.1, X1-1.S; no longer J1.2, XA1G$1.ADC.2, ☈2.2
- net SYSTWI.!INT: no longer J1.ID
- net SYSTWI.SCL: no longer J1.D-
- net SYSTWI.SDA: no longer J1.D+
- net VDD: now also X5-1.S; no longer R1.1, R3.1, R5.1
- net VIN: now also R4.2
Other:
- note added: "REWARD"
- note added: "RIPUP/PATCH QUICKFIX OPT"
- note added: "same logic with user leds if you want a blinken, DIY fgt."
- note removed: "2.4 - 3.5 V (LOW POWER!)"
- note removed: "Fix wire conflicts afterwards"
- note removed: "NOTE: Place/Route is below GYRO"
- note removed: "ROUTING"
- note removed: "Schmitt-Triggered HIGH: 2.0V to VDD"
- note removed: "TODO: Connect once final airwires are to be done since pinswap doesn't work with this symbol"
- note removed: "TODO: Default Bias on Stage 1+2 Control Signals here using pasives!"
- note removed: "TODO: GPIO to Submodules"
- note removed: "TODO: Reset Signals to submodules?"
- note removed: "TODO: Status LEDs"
- note removed: "actually, use (yet another) module for that looks nicer than a bus."
- note removed: "removed because really close to output caps of 5VDCDC"
- moved on the sheet: X2.3-1, X2.3-2

Commit message: Update Report - BaseBoard: several new exiting things!  +> finally redid SPI peripheral lines, microstripped design is superiour and easier to route  +> began working on the LED indicators to finally make the campus ee-lab guy     not talk about LED indicators for approval  +> speaking of, nearly all footprints are extra-long, should pass this time     (wasn't even that hard)  +> added a bunch of footprints regarding bus tapping points     (those footprints take board of my design, reluctantly so as it's my thing)     (will NOT be populated of course! They serve as wirepads foremost.      I will be the last person in the group to ever fill out form after     form for extra BOM approvals. Can't have nice things in times like these)  +> found the button for off-45° grid detection in the DRC, just kick me.     (now re-tracing will be a walk in the park and not tedious guess work)  +> added layer indicator near fiducial in SW/Bot corner,     (just a PCB designer thing to quickly see how many layers there are)     (copper over dimension is 100% correct, to see where the layers reside      in this sh!t sandvich of a board)  -> dropped the stupid system bus connectors in favour of my poststamp thing  -> moved OD driver unit off the board temporarily, literally the last thing     to ever worry about  -> moved FH logo from bottom to top side, ADNS sadly covers it.     (Reason: Utility > Aesthetics, see the landing pattern on bottom)     (addd: if there is time left - like hell there is - I will scale and place it somewhere on top to appease the profs =] )
 Message of the Day:

  _________________________________________
/ IGlycS9ib290c3RyYXAgbGluZSAtIFRoYW5rcyB \
\ mb3Igbm90aGluZy4K :(                    /
 -----------------------------------------
  \            .    .     .
   \      .  . .     `  ,
    \    .; .  : .' :  :  : .
     \   i..`: i` i.i.,i  i .
      \   `,--.|i |i|ii|ii|i:
           UooU\.'@@@@@@`.||'
           \__/(@@@@@@@@@@)'
                (@@@@@@@@)
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
Parts:
- removed D1: BAS40-05, diode:BAS40-05
- removed R1: 100R, rcl:R-EU_R0402
- removed SV3: (no value), con-lsta:FE05-2W
- added R10, R11, R12, R13, R14, R9: (no value), rcl:R-EU_R0201
- added X4: SYSTEMI-SW, con-hht.systewi:SYSTEWI-XR1PS08
- added X7: SYSTEMI-SE, con-hht.systewi:SYSTEWI-XR1PS08
- X3: value 87758-1016 -> SYSTEMI-CW; device con-molex:87758-1016 -> con-hht.systewi:SYSTEWI-XR1PS08
Connections:
- removed net COMP: R1.1
- removed net CTRL.A: R1.1
- removed net DDC.CLN: R1.+
- removed net DDC.VIN: R1.-
- removed net EN0: R1.2
- removed net INACT: R1.1
- removed net VDD: X5-1.S, ☈2.1
- removed net VOUT: R1.2
- removed net V~IN: D1.A
- removed net ↔BOOST: D1.C
- removed net ↔CLN: R1.K+
- removed net ↔ILIM: D1.A
- removed net ↔IN: R1.K-
- removed net ↔SENSE+: R1.K+
- removed net ↔SENSE-: R1.K-
- new net !RESET: R9.2
- new net BIAS: R11.2, R12.2
- new net CL: R9.2
- new net CTRL.!CHRG: R11.1
- new net CTRL.!FLT: R12.1
- new net CX: R10.2
- new net MRXS: PAD1.P
- new net MTXS: PAD2.P
- new net N$7: JP4.4, R12.1, R14.2
- net !CS0: no longer R1.2
- net +3V3: now also R11.2, R12.2, R9.1, X3.VCM, X4.VCM, X7.VCM; no longer JP4.2, JP4.4, R1.1
- net +4.1V: no longer R1.1
- net +5V: now also X3.VTL, X4.VTL
- net COM: no longer R1.1
- net COM.RRX: no longer R1.1
- net DDC.OUT: no longer R1.+
- net GND: now also R10.1, R13.1, R14.1, R9.1, X3.VGND, X4.VGND, X7.VGND; no longer R1.2
- net IN+&REF: no longer R1.2
- net N$1: no longer D1.C, R1.2
- net N$11: no longer D1.A2
- net N$2: now also R10.1
- net N$3: now also R9.1
- net N$4: no longer D1.A1, R1.2
- net N$5: now also R9.2
- net N$6: now also R10.2
- net N$8: now also JP4.2, R11.1, R13.2
- net SYSTWI.!INT: now also X3.!BANG, X4.!BANG, X7.!BANG
- net SYSTWI.SCL: now also X3.SCLK, X4.SCLK, X7.SCLK
- net SYSTWI.SDA: now also X3.SDAT, X4.SDAT, X7.SDAT
- net VSYS: now also X3.VBP, X4.VBP, X5-1.S, ☈2.1
- net ~SENSE+: no longer R1.-
Other:
- note added: ""its like a hub, but neither usb nor retarded like usb""
- note added: "(given the application as a ""automotive"" bus)"
- note added: "override"
- note added: "thank me later"
- note added: "todo: molex vertical micro usb -> system bus -> perph"
- note removed: "[an01]"
- moved on the sheet: JP4, R3, R4, R5

Commit message: baseboard SV2->3 (15 wires left)
Changelog:
 +> massive complexity savings in DC/DC area, I don't even know how this
    just collapsed in onto itself.
 +> added some tap footprints on back side with eventual GPIO
 -> moved out UART resistor network:
    l> false location, logically it belongs on the trackboard
    l> this entails a good amount of complexity savings regarding the
       UART receiver
    l> speaking of, I'll replace it later today with a off-the-shelf
       optocouple, like it should've been from the beginning!
    l> Seriously, why didn't they do it?
       Was it because maybe Carrera didn't do it too in their cheap design?
    l> of course, since it is an upgrade, it is an optional, the 2res net
       will remain. I'd strongly appreciate it tough that
       we use proper isolation, since the SoC is not cheap and 30V could easily creep in there someday especially when the resistors are just
       thrown in all nilly-willy
 +> LED indicator area pretty much done to death, looks nice and has even 1
    (read:ONE) user LED for indicating a failure mode.
    l> sidenote: replace with a SOT4 footprint and use pins as !RST/DAT
       Would be interesting if there is a LED with an integrated watchdog
       that starts blinking when there hasn't been activity on the
       IRQ line for a second or so. I wonder where I can buy this?
    l> turns out there's already the possibility to retrofit a neopixel
       model 8mm with the existing taps. good.
TODO:
 !> upgrade input protection using UC3610N (DIP!) as an optional.
    there's plenty of room and it's annoying that it
    can only drive in one direction all the time.
 !> add even more indicator lights, mainly in the IPC sector:
    l> also do a sidemount to make things visible.
 !> DO NOT FORGET TO ADD DUPONT CONNECTORS (F/M, F/F, M/M, whatever)
    as we will need them sooner or later for patching stuff under the
    hood so to say. est. 50mm max sound good in length?
 !> put an open collector dr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
Parts:
- removed X3: SYSTEMI-CW, con-hht.systewi:SYSTEWI-XR1PS08
- added AMO, BMO: MOTO, led:LEDCHIP-LED0805
- added R1, R15, R16: 100R, rcl:R-EU_0204/2V
- added R17: 100R, rcl:R-EU_R0201
- added R18, R19, R20: (no value), rcl:R-EU_R0201
- added X8: STMI-CW/GPIO, con-hht.systewi:SYSTEWI-XR1/PSXPS16/G8
- LED2: value VSYS -> DC3
- LED3: value 5VCC -> DC5
- LED4: value 3VCC -> SY4
- R13, R14: value (none) -> 10k/⎒; device rcl:R-EU_R0201 -> rcl:R-EU_R0402
- R8: device rcl:R-EU_R0402 -> rcl:R-EU_0204/2V
- X4, X7: device con-hht.systewi:SYSTEWI-XR1PS08 -> con-hht.systewi:SYSTEWI-XR1/PSXPS08
Connections:
- removed net N$11: R3.2, R4.2, R5.2, R6.1, R7.1
- removed net N$5: R9.2, XA1G$3.IO.7
- new net COMP: R1.1
- new net CTRL.A: R1.1
- new net DDC.CLN: R1.+
- new net DDC.VIN: R1.-
- new net EN0: R1.2
- new net INACT: R1.1
- new net N$16: LED3.A, R15.2
- new net N$31: LED4.A, R16.1
- new net N$32: LED5.A, R17.1
- new net N$33: R17.2, X4.IF.VBUS
- new net N$34: AMO.A, R18.1
- new net N$35: BMO.A, R19.1
- new net N$9: LED2.A, R1.1
- new net SYSTWI.VBUS: R20.1, R3.2, R4.2, R5.2, R6.1, R7.1, X7.IF.VBUS
- new net TOP.ODA: XA1G$3.IO.4
- new net TOP.ODB: XA1G$3.IO.7
- new net VOUT: R1.2
- new net ↔CLN: R1.K+
- new net ↔IN: R1.K-
- new net ↔SENSE+: R1.K+
- new net ↔SENSE-: R1.K-
- net !CS0: now also R1.2
- net +18V: now also R8.1
- net +3V3: now also JP4.2, JP4.4, R1.1, R1.2, R13.2, R14.2, X4.IF.VCM, X7.IF.VCM, X8.IF.VCM; no longer R11.2, R12.2, X3.VCM, X4.VCM, X7.VCM
- net +5V: now also R15.1, X4.IF.VTL, X8.IF.VTL; no longer X3.VTL, X4.VTL
- net COM: now also R1.1
- net COM.RRX: now also R1.1
- net DDC.OUT: now also R1.+
- net GND: now also AMO.C, BMO.C, LED1.C, LED2.C, LED3.C, LED4.C, LED5.C, R1.2, R11.1, R12.1, X4.IF.VGND, X7.IF.VGND, X8.IF.VGND; no longer R13.1, R14.1, X3.VGND, X4.VGND, X7.VGND
- net IN+&REF: now also R1.2
- net LAP: now also X1.2.3; no longer X1.2.4
- net N$1: now also R1.2
- net N$2: no longer R10.1
- net N$3: no longer R9.1
- net N$4: now also LED1.A, R8.2
- net N$6: now also R11.2, R13.1; no longer R10.2, XA1G$3.IO.4
- net N$7: now also R12.2, R14.1; no longer JP4.4, R12.1, R14.2
- net N$8: no longer JP4.2, R11.1, R13.2
- net PWR.MOTA: now also R19.2
- net PWR.MOTB: now also R18.2
- net SYSTWI.!INT: now also X4.IF.!BANG, X7.IF.!BANG, X8.IF.!BANG; no longer X3.!BANG, X4.!BANG, X7.!BANG
- net SYSTWI.SCL: now also X4.IF.SCLK, X7.IF.SCLK, X8.IF.SCLK; no longer X3.SCLK, X4.SCLK, X7.SCLK
- net SYSTWI.SDA: now also X4.IF.SDAT, X7.IF.SDAT, X8.IF.SDAT; no longer X3.SDAT, X4.SDAT, X7.SDAT
- net TACH: now also X1.2.4; no longer X1.2.3
- net VSYS: now also R16.2, R20.2, X4.IF.VBP, X8.IF.VBP; no longer X3.VBP, X4.VBP
- net ~SENSE+: now also R1.-
Other:
- note added: "USR"
- note removed: "thank me later"
- moved on the sheet: JP4, LED5, R10, R11, R12, R13, R14, R3, R4, R5, R6, R7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
