File: Hardware/baseboard/eagle/CarrerAI_BB_V1.0.sch (EAGLE design)
At the start: 57 parts, among them X1 JST-4POS-2X4POS, X1.2 TACH/LAP, X2.2 VRAILS+, X2.3 SoC, X4 SYSTEMI-SW, X5 87758-0816, X6 87758-0616, X7 SYSTEMI-SE, X8 STMI-CW/GPIO

Commit message: Baseboard SV3.01
Changelog:
 +> added usb again because I was bored
 +> adjusted some routes in the center
 +> I2C VBUS selector has been improved
 +> after reexamination of the cad model, there is a slack on the north
    and south side by a a few millimeters, which makes things easier.
    That's what one gets for assuming things.

Message of the Day:
 _____________________________________
/ You are not dead yet. But watch for \
\ further reports.                    /
 -------------------------------------
  \
   \
       __
      UooU\.'@@@@@@`.
      \__/(@@@@@@@@@@)
           (@@@@@@@@)
           `YY~~~~YY'
            ||    ||
Parts:
- removed JP2: (no value), pinhead:PINHD-1X1
- removed PAD1, PAD2: (no value), wirepad:1,6/0,9
- added R21, R22, R23, R24, R25, R26, R27, R28: (no value), rcl:R-EU_R0201
- added REF1: REF.EDULIMIT, kitt.refs:REF.EDULIMIT
- added SWX.1, SWX.2, SWX.3, SWX.4, SWX.5, SWX.6, SWX.7, SWX.8: (no value), wirepad:SMD2
- added U$2: 1051330011, kitt.con:1051330011
- JP1: device pinhead:PINHD-1X1 -> jumper:JP2QE
Connections:
- removed net MRXS: PAD1.P
- removed net MTXS: PAD2.P
- removed net UNO.ADC1: XA1G$1.ADC.1, ☈1.2
- removed net UNO.ADC2: XA1G$1.ADC.2, ☈2.2
- new net N$18: XA1G$1.ADC.1, ☈2.2
- new net N$19: XA1G$1.ADC.0, ☈1.2
- new net N$20: R22.1, U$2.D+
- new net N$21: R21.1, U$2.D-
- new net N$22: R23.1, R27.1, U$2.VBUS
- new net N$23: R27.2, U$2.ID
- new net N$24: R22.2, R24.2
- new net N$25: R21.2, R25.2
- net +18V: no longer JP1.1, JP2.1, PAD1.P, PAD2.P
- net GND: now also U$2.GND
Other:
- note added: "J-BEND DIL SW"
- note added: "SWx.y"
- moved on the sheet: ☈1, ☈2
