File: Hardware/baseboard/eagle/CarrerAI_BB_V1.0.sch (EAGLE design)
At the start: 72 parts, among them X1 JST-4POS-2X4POS, X1.2 TACH/LAP, X2.2 VRAILS+, X2.3 SoC, X4 SYSTEMI-SW, X5 87758-0816, X6 87758-0616, X7 SYSTEMI-SE, X8 STMI-CW/GPIO

Commit message: Baseboard v3.XYZ ---- 1. Whoever called the ambulance, thanks I guess?    Thank your lucky stars I don't have to pay up.    2.6 %/100 nothing serious. 2. Work is never over, also I am bored at the AKH Linz what else am I to do?
Message of the Morning:
 __________________________________
/ Be cheerful while you are alive. \
|                                  |
\ -- Phathotep, 24th Century B.C.  /
 ----------------------------------
 \              /\
  \             )~)
    /\/\       ( (
   ( oo )_-------_)
    \__/         )
     \/ /|/---\|\
      .. ..  ..  ..
Parts:
- removed R23, R24, R25, R26, R27, R28: (no value), rcl:R-EU_R0201
- removed SWX.1, SWX.2, SWX.3, SWX.4, SWX.5, SWX.6, SWX.7, SWX.8: (no value), wirepad:SMD2
- removed U$2: 1051330011, kitt.con:1051330011
- removed ☈1, ☈10, ☈11, ☈2, ☈3: (no value), jumper:SJ
- added JMP1, JMP2: 0R-JUMPA, jump-0r-smd:0R-JUMPA
- added L3, L6: CM CHOKE, rcl:L-EUL3216C
- added S2, S6: 219-04, switch-dil:219-04
- added S4: (no value), switch:255SB
- added S5: 9450-2, switch-misc:9450-2
- added X9: 87758-0616, con-molex:87758-0616
Connections:
- removed net CORE.ADCX: ☈10.1
- removed net CORE.ADCY: ☈11.1
- removed net N$20: R22.1, U$2.D+
- removed net N$21: R21.1, U$2.D-
- removed net N$22: R23.1, R27.1, U$2.VBUS
- removed net N$23: R27.2, U$2.ID
- removed net N$24: R22.2, R24.2
- removed net N$25: R21.2, R25.2
- removed net TOP.MVPRW: ☈3.1
- new net AUX.USB/D+_P: JMP2-0R.1
- new net AUX.USB/D-_N: JMP1-0R.1
- new net B-ID: R5.1
- new net EN/BIAS: R15.2
- new net N$17: L6.2
- new net N$5: L3.1, L6.1, R15.1, R22.2, X2.2-2.1
- new net O>D+: R22.1
- new net O>D-: R21.1
- new net OD\!SHUT: R10.1, R11.1, R7.1
- new net P=MGND: R1.2, R2.2, R3.2, R4.2, R5.2
- new net P=SGND: R1.1, R2.1, R3.1, R4.1
- new net SHUT: R7.2, X1-1.S
- new net UNO.RX: JMP1-0R.2, XA1G$3.IO.0
- new net UNO.TX: JMP2-0R.2, XA1G$3.IO.1
- new net V+: R10.2
- new net V+++: R13.2
- net +3V3: now also LED1.A, LED2.A
- net +4.1V: no longer ☈1.1
- net GND: now also L3.2, R14.1, R5.1; no longer U$2.GND, X2.2-2.1
- net N$1: now also LED2.C, R11.2, R12.1, R13.1, R16.2; no longer R7.1
- net N$18: no longer ☈2.2
- net N$19: no longer ☈1.2
- net N$2: now also LED1.C, R10.1, R10.2, R12.2, R14.2
- net N$3: now also R16.1
- net N$6: now also R21.2
- net N$8: no longer R7.2, X1-1.S
- net TOP.MTXS: now also JMP2-0R.3; no longer XA1G$3.IO.1
- net TOP.RRX: now also JMP1-0R.3; no longer XA1G$3.IO.0
- net UNO.ADC3: no longer ☈3.2
- net UNO.ADC4: no longer ☈10.2
- net UNO.ADC5: no longer ☈11.2
- net V+PWR: now also R5.2
- net VSYS: no longer ☈2.1
Other:
- note added: "Battery Guard Comparator"
- note added: "opto removed"
- note added: "«CORE»"
- note removed: "Battery Guard Circuit / Contactor"
- note removed: "J-BEND DIL SW"
- note removed: "SWx.y"
- note removed: "«SENSOR CORE»"
- moved on the sheet: R21, R22, X2-1, X2-2, X2-3, X2.2-1, X2.2-2, X5-1, X5-2, X5-3, X5-4, X5-5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
