File: Hardware/baseboard/eagle/CarrerAI_BB_V1.0.brd (EAGLE design)
At the start: 59 x 55 mm, 191 parts, among them X1 JST-4POS-2X4POS, X1.2 TACH/LAP, X2.2 VRAILS+, X2.3 SoC, X3 87758-1016, X5 87758-0816, X6 87758-0616

Commit message: Update Report - BaseBoard: several new exiting things!  +> finally redid SPI peripheral lines, microstripped design is superiour and easier to route  +> began working on the LED indicators to finally make the campus ee-lab guy     not talk about LED indicators for approval  +> speaking of, nearly all footprints are extra-long, should pass this time     (wasn't even that hard)  +> added a bunch of footprints regarding bus tapping points     (those footprints take board of my design, reluctantly so as it's my thing)     (will NOT be populated of course! They serve as wirepads foremost.      I will be the last person in the group to ever fill out form after     form for extra BOM approvals. Can't have nice things in times like these)  +> found the button for off-45° grid detection in the DRC, just kick me.     (now re-tracing will be a walk in the park and not tedious guess work)  +> added layer indicator near fiducial in SW/Bot corner,     (just a PCB designer thing to quickly see how many layers there are)     (copper over dimension is 100% correct, to see where the layers reside      in this sh!t sandvich of a board)  -> dropped the stupid system bus connectors in favour of my poststamp thing  -> moved OD driver unit off the board temporarily, literally the last thing     to ever worry about  -> moved FH logo from bottom to top side, ADNS sadly covers it.     (Reason: Utility > Aesthetics, see the landing pattern on bottom)     (addd: if there is time left - like hell there is - I will scale and place it somewhere on top to appease the profs =] )
 Message of the Day:

  _________________________________________
/ IGlycS9ib290c3RyYXAgbGluZSAtIFRoYW5rcyB \
\ mb3Igbm90aGluZy4K :(                    /
 -----------------------------------------
  \            .    .     .
   \      .  . .     `  ,
    \    .; .  : .' :  :  : .
     \   i..`: i` i.i.,i  i .
      \   `,--.|i |i|ii|ii|i:
           UooU\.'@@@@@@`.||'
           \__/(@@@@@@@@@@)'
                (@@@@@@@@)
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
Parts:
- removed D1: BAS40-05, diode:SOT23
- removed R1: 100R, rcl:R0402
- removed SV3: (no value), con-lsta:FE05-2W
- added A7:PAD1, A7:PAD2: (no value), wirepad:SMD1,27-2,54
- added R10, R11, R12, R13, R14, R9: (no value), rcl:R0201
- added X4: SYSTEMI-SW, con-hht.systewi:SYSTEWI-BR1.SOIC8C
- added X7: SYSTEMI-SE, con-hht.systewi:SYSTEWI-BR1.SOIC8C
- X3: value 87758-1016 -> SYSTEMI-CW; device con-molex:87758-1016 -> con-hht.systewi:SYSTEWI-BR1.SOIC8C
- moved R3 104.8 mm to (112.2, 11.8)
- moved R4 104.8 mm to (113.6, 11.8)
- moved R5 104.8 mm to (114.9, 11.8)
- moved R6 104.8 mm to (112.6, 13.7)
- moved R7 104.8 mm to (114.5, 13.7)
- moved U$2 52.7 mm to (56.8, 2.22)
- moved A1:R1 48.9 mm to (91.7, 15.9)
- moved A1:R2 48.9 mm to (88.1, 15.9)
- moved A1:U1 48.9 mm to (89.9, 15.9)
- moved X3 25.7 mm to (38.7, 26.0), flipped to the bottom, turned to 270 degrees
- moved A2:R2 8.77 mm to (9.53, 20.0), flipped to the bottom, turned to 180 degrees
- moved A2:R1 5.99 mm to (9.53, 22.5), flipped to the bottom, turned to 0 degrees
- moved A6:☇6 2.32 mm to (18.7, 24.8)
- moved A6:☇9 1.98 mm to (15.6, 28.7)
- moved A10:REF2 1.09 mm to (39.6, 25.8), flipped to the top, turned to 90 degrees
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Connections:
- removed net N$1: D1.3
- removed net N$4: D1.1, R1.2
- removed net VDD: A10:R4.2, A10:U1.7, A5:C2.1, A5:R3.1, A5:R4.2, A5:R5.2, A5:T1.5, A5:T1.6, A5:U1.20, A7:⌁3.P$1, A9:C1.1, A9:L1.1, A9:R4.2, A9:U1.3, X5.1, ☈2.1
- new net N$7: JP4.4, R12.1, R14.2
- new net N$8: JP4.2, R11.1, R13.2
- new net VSYS: A10:R4.2, A10:U1.7, A5:C2.1, A5:R3.1, A5:R4.2, A5:R5.2, A5:T1.5, A5:T1.6, A5:U1.20, A7:⌁3.P$1, A9:C1.1, A9:L1.1, A9:R4.2, A9:U1.3, X3.8, X4.8, X5.1, ☈2.1
- net +3V3: now also R11.2, R12.2, X3.6, X4.6, X7.6; no longer JP4.2, JP4.4
- net +4.1V: no longer R1.1
- net +5V: now also X3.7, X4.7
- net GND: now also R13.1, R14.1, X3.5, X4.5, X7.5
- net N$11: no longer D1.2
- net N$2: now also R10.1
- net N$3: now also R9.1
- net N$5: now also R9.2
- net N$6: now also R10.2
- net SYSTWI.!INT: now also X3.4, X4.4, X7.4
- net SYSTWI.SCL: now also X3.2, X4.2, X7.2
- net SYSTWI.SDA: now also X3.3, X4.3, X7.3
- net TOP.MTXS: now also A7:PAD2.1
- net TOP.RRX: now also A7:PAD1.1
Routing:
- net VSYS: track 0.00 -> 68.0 mm, vias 0 -> 21
- net VDD: track 64.8 -> 0.00 mm, vias 19 -> 0
- net GND: track 23.8 -> 82.9 mm, vias 74 -> 82
- net !CS0: track 49.3 -> 17.4 mm
- net !CS1: track 37.2 -> 5.27 mm
- net TOP.FREQ: track 7.80 -> 38.2 mm, vias 0 -> 1
- net SYSTWI.SCL: track 93.4 -> 121.7 mm, vias 1 -> 2
- net SYSTWI.SDA: track 94.0 -> 122.0 mm, vias 1 -> 2
- net +5V: track 59.1 -> 83.5 mm, vias 3 -> 4
- net SYSTWI.!INT: track 91.6 -> 76.8 mm, vias 2 -> 1
- net N$6: track 13.8 -> 0.00 mm
- net N$5: track 10.1 -> 0.00 mm, vias 1 -> 0
- net TACH: track 18.2 -> 8.61 mm
- net N$3: track 10.0 -> 0.48 mm
- net N$11: track 8.78 -> 0.00 mm
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- added copper zone on layer 15, net +5V
- added copper zone on layer 1, net VSYS
- added copper zone on layer 15, net VSYS
- added copper zone on layer 16, net VSYS
- removed copper zone on layer 1, net VDD
- removed copper zone on layer 15, net VDD
- removed copper zone on layer 16, net VDD
Other:
- board text added: "(my ip, my rules, deal with it=)"
- board text added: "0"
- board text added: "1"
- board text added: "1,4ghz"
- board text added: "1. thin out bus wires 2. place this inside"
- board text added: "2"
- board text added: "7"
- board text added: "ADD CC BY FULL/CITE"
- board text added: "LEDLEDLEDLED !!!!!!!!!!!!!!!!!! GPIO GPIO IIC"
- board text added: "PLAQUE!"
- board text added: "VCC3"
- board text added: "VCC5"
- board text added: "VDRV18"
- board text added: "VIN"
- board text added: "VSYS4"
- board text added: "X"
- board text added: "antenna danger"
- board text added: "makes a great keychain too"
- board text added: "nfets no"
- board text added: "pads"
- board text added: "reflect angles emc"
- board text added: "xnd fh board in"
- board text added: "√"
- board text removed: "3VCC"
- board text removed: "5VCC"
- board text removed: "GRADOS Generic Robotic Automation Developer Open-Hardware System"
- board text removed: "KITT evolves into"
- board text removed: "SYSTEWI"
- board text removed: "VSYS"

Commit message: baseboard SV2->3 (15 wires left)
Changelog:
 +> massive complexity savings in DC/DC area, I don't even know how this
    just collapsed in onto itself.
 +> added some tap footprints on back side with eventual GPIO
 -> moved out UART resistor network:
    l> false location, logically it belongs on the trackboard
    l> this entails a good amount of complexity savings regarding the
       UART receiver
    l> speaking of, I'll replace it later today with a off-the-shelf
       optocouple, like it should've been from the beginning!
    l> Seriously, why didn't they do it?
       Was it because maybe Carrera didn't do it too in their cheap design?
    l> of course, since it is an upgrade, it is an optional, the 2res net
       will remain. I'd strongly appreciate it tough that
       we use proper isolation, since the SoC is not cheap and 30V could easily creep in there someday especially when the resistors are just
       thrown in all nilly-willy
 +> LED indicator area pretty much done to death, looks nice and has even 1
    (read:ONE) user LED for indicating a failure mode.
    l> sidenote: replace with a SOT4 footprint and use pins as !RST/DAT
       Would be interesting if there is a LED with an integrated watchdog
       that starts blinking when there hasn't been activity on the
       IRQ line for a second or so. I wonder where I can buy this?
    l> turns out there's already the possibility to retrofit a neopixel
       model 8mm with the existing taps. good.
TODO:
 !> upgrade input protection using UC3610N (DIP!) as an optional.
    there's plenty of room and it's annoying that it
    can only drive in one direction all the time.
 !> add even more indicator lights, mainly in the IPC sector:
    l> also do a sidemount to make things visible.
 !> DO NOT FORGET TO ADD DUPONT CONNECTORS (F/M, F/F, M/M, whatever)
    as we will need them sooner or later for patching stuff under the
    hood so to say. est. 50mm max sound good in length?
 !> put an open collector dr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
Parts:
- removed A1:R1, A1:R2: 10kR/⎑, rcl:R0402
- removed A1:U1: SI1922EDH, kitt.ic:SC70-6
- removed A5:☇4, A6:☇2, A6:☇3: PTR1TP07R, testpad:TP07R
- removed U$2: (no value), marks:PASSER-CIRCLE
- removed X3: SYSTEMI-CW, con-hht.systewi:SYSTEWI-BR1.SOIC8C
- added A11:U1: 2NANDSOP8, kitt.ic:SOP65P490X110-8N
- added AMO, BMO: MOTO, led:CHIP-LED0805
- added R1, R15, R16: 100R, rcl:0204V
- added R17: 100R, rcl:R0201
- added R18, R19, R20: (no value), rcl:R0201
- added X8: STMI-CW/GPIO, con-hht.systewi:SYSTEWI-BR1.SOIC16
- A7:R1, A7:R2, A7:R3, A7:R4, A7:R5, A7:R6: device rcl:R0402 -> rcl:MINI_MELF-0102R
- A7:R8: device rcl:R0402 -> rcl:R0201
- LED2: value VSYS -> DC3
- LED3: value 5VCC -> DC5
- LED4: value 3VCC -> SY4
- R13, R14: value (none) -> 10k/⎒; device rcl:R0201 -> rcl:R0402
- R8: device rcl:R0402 -> rcl:0204V
- moved R8 145.1 mm to (9.84, 11.7), turned to 180 degrees
- moved R7 83.5 mm to (31.1, 9.84), turned to 0 degrees
- moved R5 81.9 mm to (33.2, 6.03), turned to 0 degrees
- moved R6 81.7 mm to (31.1, 7.94)
- moved R4 80.5 mm to (33.2, 7.94), turned to 0 degrees
- moved R3 79.0 mm to (33.2, 9.84), turned to 0 degrees
- moved R12 63.0 mm to (37.3, 6.35), turned to 180 degrees
- moved R11 58.8 mm to (37.5, 9.84), turned to 180 degrees
- moved R14 56.9 mm to (37.9, 7.46)
- moved R13 55.9 mm to (37.9, 8.73)
- moved A7:DCL1 44.9 mm to (63.2, 14.5)
- moved A10:REF2 32.6 mm to (71.6, 31.8)
- moved A4:R2 16.6 mm to (65.5, 46.4)
- moved A4:R1 14.6 mm to (64.5, 41.6)
- moved A7:R1 10.7 mm to (37.3, 17.1), flipped to the top, turned to 90 degrees
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Connections:
- removed net A1:COM: A1:R1.1, A1:R2.1, A1:U1.1, A1:U1.4
- removed net A7:ADC2: A7:⌁7.P$1
- removed net N$11: R3.2, R4.2, R5.2, R6.1, R7.1
- removed net N$5: A1:R2.2, A1:U1.5, R9.2, XA1.IO.7
- removed net N$8: JP4.2, R11.1, R13.2
- new net N$16: LED3.A, R15.2
- new net N$31: LED4.A, R16.1
- new net N$32: LED5.A, R17.1
- new net N$33: R17.2, X4.1
- new net N$34: AMO.A, R18.1
- new net N$35: BMO.A, R19.1
- new net N$4: LED1.A, R8.2
- new net N$9: LED2.A, R1.1
- new net SYSTWI.VBUS: R20.1, R3.2, R4.2, R5.2, R6.1, R7.1, X7.1
- new net TOP.ODA: A11:U1.1, XA1.IO.4
- new net TOP.ODB: A11:U1.6, XA1.IO.7
- new net VBP: X7.8
- new net VBUS: X8.1
- new net VTL: X7.7
- net +18V: now also R8.1
- net +3V3: now also A11:U1.8, JP4.2, JP4.4, R1.2, R13.2, R14.2, X8.6; no longer R11.2, R12.2, X3.6
- net +5V: now also R15.1, X8.7; no longer X3.7
- net A5:↔FBG: no longer A5:☇4.TP
- net GND: now also A11:U1.4, AMO.C, BMO.C, LED1.C, LED2.C, LED3.C, LED4.C, LED5.C, R11.1, R12.1, X8.5; no longer R13.1, R14.1, X3.5
- net ITH: no longer A6:☇2.TP
- net LAP: now also X1.2.3; no longer X1.2.4
- net N$2: now also A11:U1.3; no longer A1:U1.3, R10.1
- net N$3: now also A11:U1.7; no longer A1:U1.6, R9.1
- net N$6: now also A11:U1.2, R11.2, R13.1; no longer A1:R1.2, A1:U1.2, R10.2, XA1.IO.4
- net N$7: now also A11:U1.5, R12.2, R14.1; no longer JP4.4, R12.1, R14.2
- net PWR.MOTA: now also R19.2
- net PWR.MOTB: now also R18.2
- net SYSTWI.!INT: now also X8.4; no longer X3.4
- net SYSTWI.SCL: now also X8.2; no longer X3.2
- net SYSTWI.SDA: now also X8.3; no longer X3.3
- net TACH: now also X1.2.4; no longer X1.2.3
- net TOP.OS1IS2: no longer A6:☇3.TP
- net VCC/2: now also A7:⌁7.P$1
- net VSYS: now also R16.2, R20.2, X8.8; no longer X3.8
Routing:
- net +3V3: track 65.0 -> 144.9 mm, vias 10 -> 16
- net TOP.RRX: track 92.4 -> 25.0 mm, vias 2 -> 1
- net +5V: track 83.5 -> 128.6 mm, vias 4 -> 2
- net !CS0: track 17.4 -> 49.9 mm, vias 1 -> 0
- net !CS1: track 5.27 -> 35.6 mm
- net GND: track 82.9 -> 111.9 mm, vias 82 -> 80
- net SYSTWI.SDA: track 122.0 -> 93.0 mm, vias 2 -> 1
- net N$1: track 0.00 -> 28.7 mm
- net TOP.!RST: track 64.0 -> 37.9 mm
- net TOP.ODA: track 0.00 -> 24.7 mm
- net VSYS: track 68.0 -> 91.4 mm, vias 21 -> 23
- net +18V: track 46.8 -> 70.1 mm, vias 4 -> 3
- net +4.1V: track 61.8 -> 41.3 mm, vias 5 -> 4
- net SYSTWI.!INT: track 76.8 -> 92.1 mm, vias 1 -> 2
- net SYSTWI.VBUS: track 0.00 -> 13.3 mm
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- removed copper zone on layer 15, net +5V
Other:
- board size 59 x 55 mm -> 59 x 58 mm
- board text added: "'A/BMO"
- board text added: "'C3"
- board text added: "'C4"
- board text added: "'R3"
- board text added: "*alternate footprint*"
- board text added: "*option*"
- board text added: "+12"
- board text added: "3"
- board text added: "4"
- board text added: "5"
- board text added: "<<CORE>>"
- board text added: "<<GUMSHOE>>"
- board text added: "<|o_o|>"
- board text added: "CC3"
- board text added: "CC5"
- board text added: "MAGNET"
- board text added: "Outgoing working Voltage"
- board text added: "OwV SELECT"
- board text added: "SY4"
- board text added: "TODO/prio-1: finish semirough and use extension wings"
- board text added: "TODO/prio-3: add UC3610"
- board text added: "TODO: prio-2: Optocouple on TrackCore"
- board text added: "TODO: prio-S++/ARMIN: add more LEDs"
- board text added: "b"
- board text added: "dont forget"
- board text added: "rlr"
- board text added: "t"
- board text added: "ugly"
- board text removed: "1,4ghz"
- board text removed: "3V"
- board text removed: "OD"
- board text removed: "PLAQUE!"
- board text removed: "VCC3"
- board text removed: "VCC5"
- board text removed: "VDRV18"
- board text removed: "VINS"
- board text removed: "VSYS4"
- board text removed: "antenna danger"
- board text removed: "everyone sign with initials here?"
- board text removed: "idk what to put here."
- board text removed: "place tname -> "gumstick" and "core" interfaces"
- board text removed: "why?"
- board text removed: "xnd fh board in"
