File: Hardware/trackboard/eagle/trackboard.sch (EAGLE design)
At the start: 41 parts, among them Q1 BS170, U1 ADNS-3080, X9.00 RESON

Commit message: updated trackboard with revised interface
Parts:
- removed C9.03: 2.2uF, rcl:C-EUC1608
- removed C9.04, C9.05: 100nF, rcl:C-EUC0805K
- removed D9.00: RED, led:LEDCHIP-LED0805
- removed DCL1: DCL.CARRERAI, kitt.refs:DCL.CARRERAI
- removed DCL2: DCL.OSH.COPPER'5MM', kitt.refs:DCL.OSH.COPPER'5MM'
- removed J2, J3: (no value), pinhead:PINHD-1X1
- removed JP1: (no value), pinhead:PINHD-1X2
- removed Q1: BS170, transistor-fet:SST5484
- removed R1, R3, R4: 100R, rcl:R-EU_R0402
- removed R2, R9.01, R9.02: 10kR, rcl:R-EU_R0402
- removed R5: (no value), rcl:R-EU_R0805
- removed R9.13: [PPR], rcl:R-EU_R0402
- removed REF1: REF.LOGO.UASUA, kitt.refs:REF.LOGO.UASUA
- removed U1: ADNS-3080, kitt.ic:ADNS-3080
- removed X9.00: RESON, Ai_Passives:RESON
- removed ⌁1, ⌁10, ⌁11, ⌁12, ⌁13, ⌁14, ⌁15, ⌁16, ⌁17, ⌁18, ⌁19, ⌁2, ⌁20, ⌁3, ⌁4, ⌁5, ⌁6, ⌁7, ⌁8, ⌁9: SINGLEPAD40MIL, kitt.con:SINGLEPAD40MIL
Connections:
- removed net !CS0: R2.2, U1.!CS, ⌁4.P$1
- removed net !CS1: ⌁5.P$1
- removed net !INT: ⌁6.P$1
- removed net !PD: R9.01.2, U1.!PD, ⌁12.P$1
- removed net +3V3: C9.04.1, C9.05.1, D9.00.A, J3.1, JP1.1, R2.1, R9.01.1, R9.02.1, U1.OPTP, U1.VDD@1, U1.VDD@2, ⌁10.P$1
- removed net GND: C9.04.2, C9.05.2, J2.1, Q1.S, R9.13.2, U1.GND@1, U1.GND@2, ⌁11.P$1, ⌁17.P$1, ⌁9.P$1
- removed net GPIO1: ⌁14.P$1
- removed net GPIO2: ⌁15.P$1
- removed net GPIO3: ⌁16.P$1
- removed net MISO: R1.1, ⌁3.P$1
- removed net MOSI: R4.1, ⌁2.P$1
- removed net N$1: U1.GUARD, X9.00.2
- removed net N$11: D9.00.C, R9.13.1
- removed net N$2: U1.OSCOUT, X9.00.3
- removed net N$3: U1.OSCIN, X9.00.1
- removed net N$4: Q1.G, U1.LEDCTRL
- removed net N$5: C9.03.1, U1.REFC
- removed net N$6: C9.03.2, U1.REFB
- removed net N$7: Q1.D, R5.1
- removed net N$8: JP1.2, R5.2
- removed net N$9: U1.NC@3
- removed net RST: R9.02.2, U1.RESET, ⌁13.P$1
- removed net SCL: ⌁8.P$1
- removed net SCLK: R3.1, ⌁1.P$1
- removed net SDA: ⌁7.P$1
- removed net U1.MISO: R1.2, U1.MISO
- removed net U1.MOSI: R4.2, U1.MOSI
- removed net U1.SCLK: R3.2, U1.SCLK
- removed net V++: ⌁20.P$1
Other:
- note added: "LAYOUT MASTER"
- note added: "Legend: ⎒…Passive Pull-Up ⎑…Passive Pull Down ☇…Test Point ⚻…Component with kelvinized Connections ⇤…Place near IC ↦…Place away from IC ✳…High EMI Node"
- note added: "USE ONLY WITH >IMPORT EAGLE DRAWING< COMMAND"
- note removed: "[NOTE] MISO/MOSI IS A CROSS CONNECTION"
- note removed: "[TODO] PACK AS MODULE FOR EASY IMPORT INTO BASEBOARD"
- note removed: "[TODO] REVIEW"
- note removed: "[TODO] SILKSCREENING"
